File: solari-control.kicad_sch (KiCad schematic)
At the start: 11 parts

Commit message: Sch: connect expander connector.
Parts:
- added C?: 22u/50V, symbol Device:C_Polarized
- added C? (x7): 100n, symbol Device:C
- added C?: 22n, symbol Device:C
- added D? (x3): LED, symbol Device:LED
- added J? (x2): Conn_01x05, symbol Connector_Generic:Conn_01x05
- added J?: Conn_01x04, symbol Connector_Generic:Conn_01x04
- added J?: DIL8, symbol Connector_Generic:Conn_02x08_Counter_Clockwise
- added Q? (x2): AO3401A, Package_TO_SOT_SMD:SOT-23, symbol Transistor_FET:AO3401A
- added R? (x10): 470R, symbol Device:R
- added R? (x8): 10k, symbol Device:R
- added U? (x5): VO0631T, Package_SO:SOIC-8_3.9x4.9mm_P1.27mm, symbol Isolator:VO0631T
Connections:
- net GND: now also C?.2, C?.2, J?.2 (Pin_2), U?.2 (C1), U?.2 (C1), U?.2 (C1), U?.2 (C1), U?.3 (C2), U?.3 (C2), U?.3 (C2), U?.3 (C2), U?.5 (GND)
- net MISO: now also R?.1, U?.6 (VO2)
- net MOSI: now also R?.2
- net SCK: now also R?.2, R?.2
- net VCC: now also C?.1, C?.1, J?.1 (Pin_1), R?.2, U?.8 (VCC)
- net MZ: now reaches U?.1 (PD3)
- net MZ: now also R?.2
- net MP: now reaches U?.2 (PD4)
- net MP: now also R?.2
- net MPARSER: now reaches U?.32 (PD2)
- net MPARSER: now also R?.2
- net MSTROBE: now reaches U?.9 (PD5)
- net MSTROBE: now also R?.2
- new net: R?.1, U?.4 (A2) (x4)
- new net: R?.1, U?.1 (A1) (x4)
- new net: Q?.1 (G), R?.1, R?.2 (x2)
- new net: R?.2, U?.6 (VO2)
- new net: R?.2, U?.7 (VO1)
- new net 0PH: C?.2, C?.2, C?.2, J?.3 (Pin_3), J?.9 (Pin_9), U?.3 (C2), U?.5 (GND), U?.5 (GND)
- new net 0V+: C?.2, C?.2, C?.2, C?.2, J?.4 (Pin_4), U?.5 (GND), U?.5 (GND)
- new net CLOCKS: J?.3 (Pin_3), R?.1, U?.6 (VO2)
- new net CLOCKT: J?.6 (Pin_6), R?.1, U?.6 (VO2)
- new net DATOS: J?.5 (Pin_5), R?.2
- new net DATOT: J?.2 (Pin_2), R?.1, U?.7 (VO1)
- new net P: J?.8 (Pin_8), Q?.3 (D)
- new net PARSER: J?.4 (Pin_4), R?.1, U?.7 (VO1)
- new net STROBE: J?.1 (Pin_1), R?.1, U?.7 (VO1)
- new net V+: C?.1, C?.1, C?.1, C?.1, J?.3 (Pin_3), R?.2, R?.2, R?.2, U?.8 (VCC), U?.8 (VCC)
- new net VPH: C?.1, C?.1, C?.1, J?.16 (Pin_16), J?.4 (Pin_4), Q?.2 (S), Q?.2 (S), R?.1, R?.1, R?.2, R?.2, U?.8 (VCC), U?.8 (VCC)
- new net Z: J?.7 (Pin_7), Q?.3 (D)
- no-connect marks 7 -> 16
Other:
- note added: "<"
- note added: ">"
- note added: "From power supply Flap unit (MR) V+ ~ outputs"
- note added: "From power supply Logical (ML) PH ~ inputs VCC = VPH = 5V"
- note added: "S = inputs T = outputs"
- moved on the sheet: C?, D?, J?, JP?, R?, U?, Y?

Commit message: Add relay connection.
Parts:
- added C? (x2): 100n, symbol Device:C
- added Q? (x2): AO3400A, Package_TO_SOT_SMD:SOT-23, symbol Transistor_FET:AO3400A
- added R? (x4): 470R, symbol Device:R
- added R? (x3): 1k, symbol Device:R
- added R? (x2): 10k, symbol Device:R
- added TP?: TP, symbol Connector:TestPoint
- added U?: VO0631T, Package_SO:SOIC-8_3.9x4.9mm_P1.27mm, symbol Isolator:VO0631T
- C?: value 22n -> 22u
- D?: value LED -> GR
- D?: value LED -> RED
- D?: value LED -> YEL
- Y?: value Crystal -> 14.7456 MHz
Connections:
- net 0V+: now also C?.1, C?.2, Q?.2 (S), Q?.2 (S), R?.1, R?.1, U?.5 (GND)
- net GND: now also D?.1 (K), D?.1 (K), D?.1 (K), TP?.1, U?.2 (C1), U?.3 (C2)
- net V+: now also C?.1, U?.8 (VCC)
- net VDO: now reaches J?.5 (Pin_5)
- net VDO: now also J?.1 (Pin_1), C?.2
- net REL1: now reaches J?.2 (Pin_2)
- net REL1: now also Q?.3 (D)
- net REL2: now reaches J?.3 (Pin_3)
- net REL2: now also Q?.3 (D)
- net MREL1: now reaches U?.10 (PD6)
- net MREL1: now also R?.1
- net MREL2: now reaches U?.11 (PD7)
- net MREL2: now also R?.1
- net LEDG: now reaches U?.23 (PC0)
- net LEDG: now also R?.1
- net LEDY: now reaches U?.24 (PC1)
- net LEDY: now also R?.1
- net LEDR: now reaches U?.25 (PC2)
- net LEDR: now also R?.1
- net at D?.2 (A): now also R?.2 (x3)
- new net: Q?.1 (G), R?.1, R?.2 (x2)
- new net: R?.2, U?.6 (VO2)
- new net: R?.2, U?.7 (VO1)
- new net: R?.2, U?.1 (A1)
- new net: R?.2, U?.4 (A2)
- no-connect marks 16 -> 20
Other:
- note added: "From power supply Flap unit (MR) V+ ~ outputs V+ = 5V VDO = 24V"
- note added: "TODO"
- note added: "To flap unit extension card"
- note removed: "From power supply Flap unit (MR) V+ ~ outputs"
- moved on the sheet: C?, D?, J?, JP?, R?, Y?

Commit message: Add ID & IP outputs.
Parts:
- added C15: 100n, symbol Device:C
- added H1, H2, H3, H4: MH, symbol Mechanical:MountingHole
- added Q5, Q6: BC327, Package_TO_SOT_THT:TO-92_Inline, symbol Transistor_BJT:BC327
- added R29, R33: 470R, symbol Device:R
- added R30, R32: 1k, symbol Device:R
- added R31, R34: 10k, symbol Device:R
- added U8: VO0631T, Package_SO:SOIC-8_3.9x4.9mm_P1.27mm, symbol Isolator:VO0631T
- gave numbers to parts that had none: 67
Connections:
- net 0V+: now also C15.2, R31.2, R34.2, U8.5 (GND)
- net GND: now also U8.2 (C1), U8.3 (C2)
- net V+: now also C15.1, Q5.3 (E), Q6.3 (E), U8.8 (VCC)
- net MID: now reaches U2.26 (PC3)
- net MID: now also R29.2
- net MIP: now reaches U2.27 (PC4)
- net MIP: now also R33.2
- net IP: now reaches J4.14 (Pin_14)
- net IP: now also Q6.1 (C), R34.1
- net ID: now reaches J4.15 (Pin_15)
- net ID: now also Q5.1 (C), R31.1
- new net: R33.1, U8.4 (A2)
- new net: Q5.2 (B), R30.1
- new net: R29.1, U8.1 (A1)
- new net: R32.2, U8.6 (VO2)
- new net: R30.2, U8.7 (VO1)
- new net: Q6.2 (B), R32.1
- no-connect marks 20 -> 24
Other:
- note added: "To parent device"
- note added: "To relay board (side switching)"
- note removed: "TODO"
- moved on the sheet: C1, C10, C11, C12, C13, C14, C2, C3, C4, C5, C6, C7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

Commit message: Use proper capacitors.
Parts:
- removed C1: 22u/50V, symbol Device:C_Polarized
- C12: value 22u -> 22u/25V
- C2: value 100n -> 22u/25V
- C3: value 100n -> 100n/50V
Other:
- moved on the sheet: C2
Changed lines of the file:
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@@
   (junction (at 74.295 267.335) (diameter 0) (color 0 0 0 0)
   )
-  (junction (at 247.015 87.63) (diameter 0) (color 0 0 0 0)
-  )
   (junction (at 85.725 101.6) (diameter 0) (color 0 0 0 0)
   )
@@
   (junction (at 98.425 58.42) (diameter 0) (color 0 0 0 0)
   )
-  (junction (at 247.015 80.01) (diameter 0) (color 0 0 0 0)
-  )
   (junction (at 98.425 187.96) (diameter 0) (color 0 0 0 0)
   )
@@
   (junction (at 130.175 44.45) (diameter 0) (color 0 0 0 0)
   )
-  (junction (at 230.505 80.01) (diameter 0) (color 0 0 0 0)
-  )
   (junction (at 230.505 59.055) (diameter 0) (color 0 0 0 0)
   )
@@
   (junction (at 199.39 162.56) (diameter 0) (color 0 0 0 0)
   )
+  (junction (at 230.505 80.01) (diameter 0) (color 0 0 0 0)
+  )
   (junction (at 98.425 93.98) (diameter 0) (color 0 0 0 0)
   )
@@
   (junction (at 73.66 227.965) (diameter 0) (color 0 0 0 0)
   )
+  (junction (at 251.206 87.63) (diameter 0) (color 0 0 0 0)
+  )
   (junction (at 346.075 97.155) (diameter 0) (color 0 0 0 0)
   )
@@
     (stroke (width 0) (type default) (color 0 0 0 0))
   )
-  (wire (pts (xy 252.73 80.01) (xy 247.015 80.01))
-    (stroke (width 0) (type default) (color 0 0 0 0))
-  )
   (wire (pts (xy 199.39 154.94) (xy 187.96 154.94))
     (stroke (width 0) (type default) (color 0 0 0 0))
@@
     (stroke (width 0) (type default) (color 0 0 0 0))
   )
-  (wire (pts (xy 247.015 80.01) (xy 230.505 80.01))
+  (wire (pts (xy 223.52 80.01) (xy 230.505 80.01))
     (stroke (width 0) (type default) (color 0 0 0 0))
   )
@@
     (stroke (width 0) (type default) (color 0 0 0 0))
   )
+  (wire (pts (xy 230.505 80.01) (xy 237.49 80.01))
+    (stroke (width 0) (type default) (color 0 0 0 0))
+  )
   (wire (pts (xy 375.285 97.155) (xy 364.49 97.155))
     (stroke (width 0) (type default) (color 0 0 0 0))
@@
     (stroke (width 0) (type default) (color 0 0 0 0))
   )
-  (wire (pts (xy 230.505 80.01) (xy 223.52 80.01))
-    (stroke (width 0) (type default) (color 0 0 0 0))
-  )
   (wire (pts (xy 107.95 241.935) (xy 98.425 241.935))
     (stroke (width 0) (type default) (color 0 0 0 0))
@@
     (stroke (width 0) (type default) (color 0 0 0 0))
   )
-  (wire (pts (xy 247.015 87.63) (xy 230.505 87.63))
+  (wire (pts (xy 230.505 87.63) (xy 251.206 87.63))
     (stroke (width 0) (type default) (color 0 0 0 0))
   )
@@
     (stroke (width 0) (type default) (color 0 0 0 0))
   )
-  (wire (pts (xy 252.73 87.63) (xy 247.015 87.63))
+  (wire (pts (xy 252.73 87.63) (xy 251.206 87.63))
     (stroke (width 0) (type default) (color 0 0 0 0))
   )
@@
     )
   )
-  (global_label "V+" (shape input) (at 252.73 80.01 0) (fields_autoplaced)
+  (global_label "V+" (shape input) (at 237.49 80.01 0) (fields_autoplaced)
     (effects (font (size 1.27 1.27)) (justify left))
-    (property "Intersheet References" "${INTERSHEET_REFS}" (id 0) (at 257.8041 79.9306 0)
+    (property "Intersheet References" "${INTERSHEET_REFS}" (id 0) (at 242.5641 79.9306 0)
       (effects (font (size 1.27 1.27)) (justify left) hide)
     )
@@
     (pin "8")
   )
-  (symbol (lib_id "Device:C_Polarized") (at 230.505 83.82 0) (mirror y) (unit 1)
-    (in_bom yes) (on_board yes)
-    (property "Reference" "C1" (id 0) (at 233.045 83.185 0)
-      (effects (font (size 1.27 1.27)) (justify right))
-    )
-    (property "Value" "22u/50V" (id 1) (at 233.045 85.09 0)
-      (effects (font (size 1.27 1.27)) (justify right))
-    )
-    (property "Footprint" "" (id 2) (at 229.5398 87.63 0)
-      (effects (font (size 1.27 1.27)) hide)
-    )
-    (property "Datasheet" "~" (id 3) (at 230.505 83.82 0)
-      (effects (font (size 1.27 1.27)) hide)
-    )
-    (pin "1")
-    (pin "2")
-  )
   (symbol (lib_id "power:GND") (at 177.8 167.64 0) (mirror y) (unit 1)
     (in_bom yes) (on_board yes) (fields_autoplaced)
@@
     (pin "3")
   )
-  (symbol (lib_id "Device:C") (at 247.015 83.82 0) (mirror y) (unit 1)
+  (symbol (lib_id "Device:C") (at 230.505 83.82 0) (mirror y) (unit 1)
     (in_bom yes) (on_board yes)
-    (property "Reference" "C2" (id 0) (at 249.555 83.185 0)
+    (property "Reference" "C2" (id 0) (at 233.045 83.185 0)
       (effects (font (size 1.27 1.27)) (justify right))
     )
-    (property "Value" "100n" (id 1) (at 249.555 85.09 0)
+    (property "Value" "22u/25V" (id 1) (at 233.045 85.09 0)
       (effects (font (size 1.27 1.27)) (justify right))
     )
-    (property "Footprint" "" (id 2) (at 246.0498 87.63 0)
+    (property "Footprint" "" (id 2) (at 229.5398 87.63 0)
       (effects (font (size 1.27 1.27)) hide)
     )
-    (property "Datasheet" "~" (id 3) (at 247.015 83.82 0)
+    (property "Datasheet" "~" (id 3) (at 230.505 83.82 0)
       (effects (font (size 1.27 1.27)) hide)
     )
@@
     (pin "2")
   )
-  (symbol (lib_id "power:PWR_FLAG") (at 247.015 87.63 180) (unit 1)
+  (symbol (lib_id "power:PWR_FLAG") (at 251.206 87.63 180) (unit 1)
     (in_bom yes) (on_board yes) (fields_autoplaced)
-    (property "Reference" "#FLG02" (id 0) (at 247.015 89.535 0)
+    (property "Reference" "#FLG02" (id 0) (at 251.206 89.535 0)
       (effects (font (size 1.27 1.27)) hide)
     )
-    (property "Value" "PWR_FLAG" (id 1) (at 247.015 92.0734 0))
-    (property "Footprint" "" (id 2) (at 247.015 87.63 0)
+    (property "Value" "PWR_FLAG" (id 1) (at 251.206 92.0734 0))
+    (property "Footprint" "" (id 2) (at 251.206 87.63 0)
       (effects (font (size 1.27 1.27)) hide)
     )
-    (property "Datasheet" "~" (id 3) (at 247.015 87.63 0)
+    (property "Datasheet" "~" (id 3) (at 251.206 87.63 0)
       (effects (font (size 1.27 1.27)) hide)
     )
@@
       (effects (font (size 1.27 1.27)) (justify left))
     )
-    (property "Value" "22u" (id 1) (at 233.68 36.195 0)
+    (property "Value" "22u/25V" (id 1) (at 233.68 36.195 0)
       (effects (font (size 1.27 1.27)) (justify left))
     )
@@
       (effects (font (size 1.27 1.27)) (justify right))
     )
-    (property "Value" "100n" (id 1) (at 233.045 92.71 0)
+    (property "Value" "100n/50V" (id 1) (at 233.045 92.71 0)
       (effects (font (size 1.27 1.27)) (justify right))
     )
@@
       (reference "#PWR019") (unit 1) (value "GND") (footprint "")
     )
-    (path "/13a0ef12-5ffc-4ee0-a989-51c38dc0f48c"
-      (reference "C1") (unit 1) (value "22u/50V") (footprint "")
-    )
     (path "/4a011d26-96c7-4c0a-841d-6bc5b1f373ce"
-      (reference "C2") (unit 1) (value "100n") (footprint "")
+      (reference "C2") (unit 1) (value "22u/25V") (footprint "")
     )
     (path "/ff5bae46-5f92-49b2-8aa4-c2b219f51ab9"
-      (reference "C3") (unit 1) (value "100n") (footprint "")
+      (reference "C3") (unit 1) (value "100n/50V") (footprint "")
     )
     (path "/818c281e-1097-4688-a9dd-901329295d04"
@@
     )
     (path "/e41b6f02-b07d-47ba-9515-15ecb6256f96"
-      (reference "C12") (unit 1) (value "22u") (footprint "")
+      (reference "C12") (unit 1) (value "22u/25V") (footprint "")
     )
     (path "/d01be9e7-bb0a-443c-a037-d17e83b89f89"
