File: solari-control.kicad_sch (KiCad schematic)
At the start: 80 parts, among them J1 Conn_01x05, J2 AVR-ISP-6, J3 Conn_01x04, J4 DIL8, J5 Conn_01x04, J6 Conn_01x05, Q1 AO3401A, Q2 AO3401A, Q3 AO3400A, Q4 AO3400A, Q5 BC327, Q6 BC327, U1 VO0631T, U2 ATmega328P-A, U3 VO0631T, U4 VO0631T, U5 VO0631T, U6 VO0631T, U7 VO0631T, U8 VO0631T, Y1 14.7456 MHz

Commit message: Add voltage levels (measured).
Other:
- note added: "From power supply Flap unit (MR) V+ ~ outputs V+ = 5V VDO = VR = 24V"
- note added: "From power supply Logical (ML) PH ~ inputs VCC = 5V VPH = 15V"
- note removed: "From power supply Flap unit (MR) V+ ~ outputs V+ = 5V VDO = 24V"
- note removed: "From power supply Logical (ML) PH ~ inputs VCC = VPH = 5V"
Changed lines of the file:
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@@
     (effects (font (size 1.27 1.27)) (justify right bottom))
   )
-  (text "From power supply\nFlap unit (MR)\nV+ ~ outputs\nV+ = 5V\nVDO = 24V"
-    (at 217.805 103.505 180)
+  (text "From power supply\nFlap unit (MR)\nV+ ~ outputs\nV+ = 5V\nVDO = VR = 24V"
+    (at 217.17 103.505 180)
     (effects (font (size 1.27 1.27)) (justify right bottom))
   )
@@
     (effects (font (size 1.27 1.27)) (justify right bottom))
   )
-  (text "From power supply\nLogical (ML)\nPH ~ inputs\nVCC = VPH = 5V"
-    (at 218.44 36.83 180)
+  (text "From power supply\nLogical (ML)\nPH ~ inputs\nVCC = 5V\nVPH = 15V"
+    (at 217.17 36.83 180)
     (effects (font (size 1.27 1.27)) (justify right bottom))
   )

Commit message: Add fuses on power input.
Parts:
- added F1, F2, F3, F4: 200mA, symbol Device:Fuse
- R3: value 470R -> 1k
Connections:
- net V+: now also F3.1, F3.2
- net VCC: now also F1.1, F1.2
- net VDO: now also F4.1, F4.2
- net VPH: now also F2.1, F2.2
Other:
- note added: "15V"
- moved on the sheet: C12, C14, C2, C3

Commit message: Add transistors for 15V outputs.
Parts:
- added C1: 10u, symbol Device:C
- added Q10, Q7, Q8, Q9: AO3400A, Package_TO_SOT_SMD:SOT-23, symbol Transistor_FET:AO3400A
- added R35, R37: 470R, symbol Device:R
- added R36, R38, R39, R40: 10k, symbol Device:R
- added U9: L78L05_SOT89, Package_TO_SOT_SMD:SOT-89-3, symbol Regulator_Linear:L78L05_SOT89
- C14: value 100n -> 22u/25V
Connections:
- net 0PH: now also C1.2, Q10.2 (S), Q7.2 (S), Q8.2 (S), Q9.2 (S), R36.1, R38.1, R39.1, R40.1, U9.2 (GND)
- net CLOCKS: now also R8.2, Q8.3 (D); no longer R8.1, U3.6 (VO2)
- net PARSER: now also R6.2, Q7.3 (D); no longer R6.1, U3.7 (VO1)
- net VPH: now also R6.1, R8.1, U9.3 (IN); no longer C8.1, C9.1, R6.2, R8.2, U3.8 (VCC), U4.8 (VCC)
- net at Q1.1 (G), R11.2: now also Q10.3 (D); no longer R13.1
- net at Q2.1 (G), R14.2: now also Q9.3 (D); no longer R15.1
- new net: Q10.1 (G), R15.1, R40.2
- new net: Q7.1 (G), R35.1, R36.2
- new net: R35.2, U3.7 (VO1)
- new net: R37.2, U3.6 (VO2)
- new net: Q9.1 (G), R13.1, R39.2
- new net: Q8.1 (G), R37.1, R38.2
- new net 5VPH: C1.1, C8.1, C9.1, U3.8 (VCC), U4.8 (VCC), U9.1 (OUT)
Other:
- moved on the sheet: C10, C11, C12, C13, C14, C15, C2, C3, C4, C5, C6, C7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

Commit message: Add footprints.
Parts:
- C1, C10, C11, C12, C13, C14, C15, C2, C3, C4, C5, C6, C7, C8, C9: footprint (none) -> Capacitor_SMD:C_0805_2012Metric_Pad1.18x1.45mm_HandSolder
- D1, D2, D4: footprint (none) -> LED_SMD:LED_0805_2012Metric_Pad1.15x1.40mm_HandSolder
- D3: footprint Package_TO_SOT_SMD:SOT-23-6 -> Package_TO_SOT_SMD:SOT-23-6_Handsoldering
- F1, F2, F3, F4: footprint (none) -> Fuse:Fuse_1206_3216Metric_Pad1.42x1.75mm_HandSolder
- H1, H2, H3, H4: footprint (none) -> MountingHole:MountingHole_3mm_Pad_Via
- J1: value Conn_01x05 -> A5081WR-5P; footprint (none) -> TerminalBlock:TerminalBlock_bornier-5_P5.08mm
- J2: footprint (none) -> Connector_PinHeader_2.54mm:PinHeader_2x03_P2.54mm_Vertical
- J3, J5: footprint (none) -> Connector_PinHeader_2.54mm:PinHeader_1x04_P2.54mm_Vertical
- J4: footprint (none) -> Package_DIP:DIP-16_W7.62mm_LongPads
- J6: value Conn_01x05 -> A5081WV-5P; footprint (none) -> TerminalBlock:TerminalBlock_bornier-5_P5.08mm
- JP1: footprint (none) -> Jumper:SolderJumper-2_P1.3mm_Open_RoundedPad1.0x1.5mm
- JP2: footprint (none) -> Connector_PinHeader_2.54mm:PinHeader_1x02_P2.54mm_Vertical
- R1, R10, R11, R12, R13, R14, R15, R16, R17, R18, R19, R2, R20, R21, R22, R23, R24, R25, R26, R27, R28, R29, R3, R30, R31, R32, R33, R34, R35, R36, R37, R38, R39, R4, R40, R5, R6, R7, R8, R9: footprint (none) -> Resistor_SMD:R_0805_2012Metric_Pad1.20x1.40mm_HandSolder
- TP1: footprint (none) -> TestPoint:TestPoint_Loop_D3.50mm_Drill1.4mm_Beaded
- Y1: footprint (none) -> Crystal:Crystal_HC49-U_Vertical

Commit message: Fix transistors on outputs.
Parts:
- removed C11, C9: 100n, Capacitor_SMD:C_0805_2012Metric_Pad1.18x1.45mm_HandSolder, symbol Device:C
- removed Q3, Q7, Q8, Q9: AO3400A, Package_TO_SOT_SMD:SOT-23, symbol Transistor_FET:AO3400A
- removed Q5, Q6: BC327, Package_TO_SOT_THT:TO-92_Inline, symbol Transistor_BJT:BC327
- removed R11, R14, R19, R26, R36, R38: 10k, Resistor_SMD:R_0805_2012Metric_Pad1.20x1.40mm_HandSolder, symbol Device:R
- removed R24, R35, R37: 470R, Resistor_SMD:R_0805_2012Metric_Pad1.20x1.40mm_HandSolder, symbol Device:R
- removed U4, U6: VO0631T, Package_SO:SOIC-8_3.9x4.9mm_P1.27mm, symbol Isolator:VO0631T
- added D2, D3: 1N4148, Diode_SMD:D_0805_2012Metric_Pad1.15x1.40mm_HandSolder, symbol Diode:1N4148
- added Q1, Q11, Q3, Q7, Q8, Q9: AO3401A, Package_TO_SOT_SMD:SOT-23, symbol Transistor_FET:AO3401A
- added Q12, Q2: AO3400A, Package_TO_SOT_SMD:SOT-23, symbol Transistor_FET:AO3400A
- added R10, R44: 100R, Resistor_SMD:R_0805_2012Metric_Pad1.20x1.40mm_HandSolder, symbol Device:R
- added R12, R13, R17, R18, R3, R31, R34, R4, R42, R43, R46, R7, R9: 10k, Resistor_SMD:R_0805_2012Metric_Pad1.20x1.40mm_HandSolder, symbol Device:R
- added U10, U11, U4, U5: PC817, Package_DIP:DIP-4_W8.89mm_SMDSocket_LongPads, symbol Isolator:PC817
- R14: renamed from R13; value 470R -> 100R
- R19: renamed from R15; value 470R -> 100R
- R21: value 470R -> 10k
- R33: renamed from R30; value 1k -> 100R
- R35: renamed from R32; value 1k -> 100R
- R40, R6: value 10k -> 100R
- renumbered C5 to C1, C6 to C10, C7 to C11, C13 to C12, C15 to C13, C12 to C2, C14 to C3, C1 to C4, C8 to C5, C2 to C6, C3 to C7, C4 to C8, C10 to C9, D3 to D1, D1 to D4, D2 to D5, D4 to D6, J3 to J1, J6 to J2, J1 to J3, J2 to J4, J4 to J5, J5 to J6, JP2 to JP1, JP1 to JP2, Q2 to Q5, Q1 to Q6, R2 to R1, R9 to R11, R12 to R15, R1 to R16, R3 to R2, R16 to R20, R17 to R22, R18 to R23, R22 to R24, R23 to R25, R4 to R26, R5 to R27, R10 to R28, R27 to R29, R28 to R30, R29 to R32, R31 to R36, R33 to R37, R34 to R38, R20 to R41, R25 to R45, R7 to R5, U9 to U2, U5 to U6, U2 to U7, U7 to U8, U8 to U9
Connections:
- net 0PH: now also R21.1, D2.2 (A), D3.2 (A), R18.1, U4.3, U5.3; no longer C5.2, Q10.2 (S), R39.1, R40.1, U3.5 (GND)
- net 0V+: now also Q10.2 (S), Q12.2 (S), R43.1, R46.1, U10.3, U11.3; no longer Q4.2 (S)
- net 5VPH: now also R8.1, Q1.2 (S), Q3.2 (S), R4.1
- net CLOCKS: now also Q4.3 (D), R7.1; no longer R8.2
- net GND: now also U10.2, U11.2, U4.2, U5.2
- net ID: now also Q7.3 (D)
- net IP: now also Q8.3 (D)
- net P: now also D2.1 (K), R18.2
- net PARSER: now also Q2.3 (D), R3.1; no longer R6.2
- net REL1: now also Q10.3 (D)
- net REL2: now also Q12.3 (D); no longer Q4.3 (D)
- net V+: now also Q7.2 (S), Q8.2 (S), R31.2, R34.1
- net VDO: now also R39.1, Q11.2 (S), Q9.2 (S), R42.1
- net VPH: now also C5.2, Q4.2 (S), U3.5 (GND), Q2.2 (S), R12.1, R13.1, R17.1, R3.2, R7.2, R9.1; no longer R6.1, R8.1
- net Z: now also R21.2, D3.1 (K)
- net at Q4.1 (G): now also Q3.3 (D), R12.2
- net at U3.7 (VO1): now also R6.2
- net at R33.1: now also Q7.1 (G), R31.1
- net at Q6.1 (G): now also R19.1, R17.2; no longer Q10.3 (D)
- net at R15.1: now also U4.1
- net at R20.1: now also U5.1
- net at R19.2: now also U5.4
- net at R14.2: now also U4.4
- net at U3.6 (VO2): now also R10.2
- net at Q5.1 (G): now also R14.1, R13.2
- net at R39.2: now also R40.1, Q9.1 (G); no longer R14.1
- net at R35.1: now also Q8.1 (G), R34.2
- net at R41.2: now also U10.1
- net at R45.2: now also U11.1
- new net: Q3.1 (G), R10.1, R8.2
- new net: R40.2, U10.4
- new net: Q1.1 (G), R4.2, R6.1
- new net: Q11.3 (D), Q12.1 (G), R46.2
- new net: Q11.1 (G), R42.2, R44.1
- new net: R44.2, U11.4
- new net: Q10.1 (G), Q9.3 (D), R43.2
- new net: Q1.3 (D), Q2.1 (G), R9.2
Other:
- moved on the sheet: C1, C10, C11, C12, C13, C2, C3, C4, C5, C6, C7, C8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

Commit message: Use 3V3 power supply.
Parts:
- added C14: 10u, Capacitor_SMD:C_0805_2012Metric_Pad1.18x1.45mm_HandSolder, symbol Device:C
- added U12: AMS1117-3.3, Package_TO_SOT_SMD:SOT-223-3_TabPin2, symbol Regulator_Linear:AMS1117-3.3
Connections:
- net GND: now also C14.2, U12.1 (GND)
- net VCC: now also C14.1, U12.2 (VO); no longer C2.1, F1.1, F1.2, J2.1 (Pin_1)
- net VDO: now also R42.2; no longer R42.1
- net at Q11.1 (G), R44.1: now also R42.1; no longer R42.2
- new net: F1.1, J2.1 (Pin_1)
- new net: C2.1, F1.2, U12.3 (VI)
Other:
- note added: "Parent device has 3.3V UART."
- moved on the sheet: C10, C11, C2, C8, F1, R42, U7, Y1

Commit message: Add power jumper for AVR-ISP connector.
Parts:
- removed JP2: SJ2O, Jumper:SolderJumper-2_P1.3mm_Open_RoundedPad1.0x1.5mm, symbol Jumper:SolderJumper_2_Open
- added JP2: Jumper_3_Open, Connector_PinHeader_2.54mm:PinHeader_1x03_P2.54mm_Vertical, symbol Jumper:Jumper_3_Open
Connections:
- net VCC: now also JP2.1 (A)
- net 5V: now reaches F1.1, J2.1 (Pin_1)
- net 5V: now also JP2.3 (B)
- net at J4.2 (VCC): now also JP2.2 (C)
Changed lines of the file:
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@@
   (junction (at 297.815 30.48) (diameter 0) (color 0 0 0 0)
   )
-  (junction (at 346.075 97.155) (diameter 0) (color 0 0 0 0)
+  (junction (at 346.075 93.345) (diameter 0) (color 0 0 0 0)
   )
   (junction (at 125.095 161.925) (diameter 0) (color 0 0 0 0)
@@
     (stroke (width 0) (type default) (color 0 0 0 0))
   )
+  (wire (pts (xy 381.635 93.345) (xy 387.985 93.345))
+    (stroke (width 0) (type default) (color 0 0 0 0))
+  )
   (wire (pts (xy 292.1 52.705) (xy 297.815 52.705))
     (stroke (width 0) (type default) (color 0 0 0 0))
@@
     (stroke (width 0) (type default) (color 0 0 0 0))
   )
-  (wire (pts (xy 346.075 97.155) (xy 346.075 102.235))
+  (wire (pts (xy 346.075 93.345) (xy 346.075 102.235))
     (stroke (width 0) (type default) (color 0 0 0 0))
   )
@@
     (stroke (width 0) (type default) (color 0 0 0 0))
   )
-  (wire (pts (xy 375.285 97.155) (xy 364.49 97.155))
-    (stroke (width 0) (type default) (color 0 0 0 0))
-  )
   (wire (pts (xy 131.445 146.685) (xy 131.445 156.845))
     (stroke (width 0) (type default) (color 0 0 0 0))
   )
-  (wire (pts (xy 356.87 97.155) (xy 346.075 97.155))
-    (stroke (width 0) (type default) (color 0 0 0 0))
-  )
   (wire (pts (xy 116.84 260.985) (xy 120.65 260.985))
     (stroke (width 0) (type default) (color 0 0 0 0))
@@
     (stroke (width 0) (type default) (color 0 0 0 0))
   )
-  (wire (pts (xy 346.075 95.25) (xy 346.075 97.155))
+  (wire (pts (xy 346.075 91.44) (xy 346.075 93.345))
     (stroke (width 0) (type default) (color 0 0 0 0))
   )
@@
     (stroke (width 0) (type default) (color 0 0 0 0))
   )
+  (wire (pts (xy 346.075 93.345) (xy 368.935 93.345))
+    (stroke (width 0) (type default) (color 0 0 0 0))
+  )
   (wire (pts (xy 165.1 250.825) (xy 160.655 250.825))
     (stroke (width 0) (type default) (color 0 0 0 0))
@@
     (effects (font (size 1.27 1.27)) (justify right bottom))
   )
+  (label "5V" (at 239.395 41.91 0)
+    (effects (font (size 1.27 1.27)) (justify left bottom))
+  )
   (label "P" (at 68.58 107.315 0)
     (effects (font (size 1.27 1.27)) (justify left bottom))
@@
     )
   )
+  (global_label "5V" (shape input) (at 387.985 93.345 0) (fields_autoplaced)
+    (effects (font (size 1.27 1.27)) (justify left))
+    (property "Intersheet References" "${INTERSHEET_REFS}" (id 0) (at 392.6962 93.2656 0)
+      (effects (font (size 1.27 1.27)) (justify left) hide)
+    )
+  )
   (global_label "MOSI" (shape input) (at 254 151.13 180) (fields_autoplaced)
     (effects (font (size 1.27 1.27)) (justify right))
@@
     (pin "1")
   )
+  (symbol (lib_id "Jumper:Jumper_3_Open") (at 375.285 93.345 0) (unit 1)
+    (in_bom yes) (on_board yes) (fields_autoplaced)
+    (property "Reference" "JP2" (id 0) (at 375.285 88.273 0))
+    (property "Value" "Jumper_3_Open" (id 1) (at 375.285 90.8099 0))
+    (property "Footprint" "Connector_PinHeader_2.54mm:PinHeader_1x03_P2.54mm_Vertical" (id 2) (at 375.285 93.345 0)
+      (effects (font (size 1.27 1.27)) hide)
+    )
+    (property "Datasheet" "~" (id 3) (at 375.285 93.345 0)
+      (effects (font (size 1.27 1.27)) hide)
+    )
+    (pin "1")
+    (pin "2")
+    (pin "3")
+  )
   (symbol (lib_id "Device:R") (at 95.25 86.995 180) (unit 1)
     (in_bom yes) (on_board yes)
@@
     (pin "3")
   )
-  (symbol (lib_id "power:VCC") (at 346.075 95.25 0) (mirror y) (unit 1)
+  (symbol (lib_id "power:VCC") (at 346.075 91.44 0) (mirror y) (unit 1)
     (in_bom yes) (on_board yes) (fields_autoplaced)
-    (property "Reference" "#PWR08" (id 0) (at 346.075 99.06 0)
+    (property "Reference" "#PWR08" (id 0) (at 346.075 95.25 0)
       (effects (font (size 1.27 1.27)) hide)
     )
-    (property "Value" "VCC" (id 1) (at 344.678 94.4138 0)
+    (property "Value" "VCC" (id 1) (at 344.678 90.6038 0)
       (effects (font (size 1.27 1.27)) (justify left))
     )
-    (property "Footprint" "" (id 2) (at 346.075 95.25 0)
+    (property "Footprint" "" (id 2) (at 346.075 91.44 0)
       (effects (font (size 1.27 1.27)) hide)
     )
-    (property "Datasheet" "" (id 3) (at 346.075 95.25 0)
+    (property "Datasheet" "" (id 3) (at 346.075 91.44 0)
       (effects (font (size 1.27 1.27)) hide)
     )
@@
     (pin "2")
   )
-  (symbol (lib_id "Jumper:SolderJumper_2_Open") (at 360.68 97.155 0) (mirror y) (unit 1)
-    (in_bom yes) (on_board yes) (fields_autoplaced)
-    (property "Reference" "JP2" (id 0) (at 360.68 92.5662 0))
-    (property "Value" "SJ2O" (id 1) (at 360.68 95.1031 0))
-    (property "Footprint" "Jumper:SolderJumper-2_P1.3mm_Open_RoundedPad1.0x1.5mm" (id 2) (at 360.68 97.155 0)
-      (effects (font (size 1.27 1.27)) hide)
-    )
-    (property "Datasheet" "~" (id 3) (at 360.68 97.155 0)
-      (effects (font (size 1.27 1.27)) hide)
-    )
-    (pin "1")
-    (pin "2")
-  )
   (symbol (lib_id "Device:R") (at 160.02 150.495 90) (unit 1)
     (in_bom yes) (on_board yes) (fields_autoplaced)
@@
       (reference "JP1") (unit 1) (value "J2O") (footprint "Connector_PinHeader_2.54mm:PinHeader_1x02_P2.54mm_Vertical")
     )
-    (path "/8ca6fc72-59cf-4423-aa66-71c8b0d90f32"
-      (reference "JP2") (unit 1) (value "SJ2O") (footprint "Jumper:SolderJumper-2_P1.3mm_Open_RoundedPad1.0x1.5mm")
+    (path "/2e19d23c-fbb7-4873-83d6-f60a7378caae"
+      (reference "JP2") (unit 1) (value "Jumper_3_Open") (footprint "Connector_PinHeader_2.54mm:PinHeader_1x03_P2.54mm_Vertical")
     )
     (path "/bede9112-c3f5-49ce-94e2-91488e69f456"

Commit message: ATmega328p: connecrt also AVCC (required by ICSP).
Parts:
- added C?: 100n, Capacitor_SMD:C_0805_2012Metric_Pad1.18x1.45mm_HandSolder, symbol Device:C
Connections:
- net GND: now also C?.2
- net VCC: now also U7.18 (AVCC), C?.1
- no-connect marks 24 -> 23
Changed lines of the file:
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@@
   (junction (at 95.25 90.805) (diameter 0) (color 0 0 0 0)
   )
+  (junction (at 299.085 146.685) (diameter 0) (color 0 0 0 0)
+  )
   (junction (at 346.075 114.935) (diameter 0) (color 0 0 0 0)
   )
@@
   (junction (at 118.11 63.5) (diameter 0) (color 0 0 0 0)
   )
+  (junction (at 299.085 133.985) (diameter 0) (color 0 0 0 0)
+  )
   (junction (at 83.82 222.885) (diameter 0) (color 0 0 0 0)
   )
@@
   (no_connect (at 258.445 179.07))
   (no_connect (at 37.465 136.525))
-  (no_connect (at 271.145 135.89))
   (no_connect (at 238.76 83.82))
   (no_connect (at 351.155 50.8))
@@
     (stroke (width 0) (type default) (color 0 0 0 0))
   )
+  (wire (pts (xy 304.8 146.685) (xy 299.085 146.685))
+    (stroke (width 0) (type default) (color 0 0 0 0))
+  )
   (wire (pts (xy 120.015 121.92) (xy 132.08 121.92))
     (stroke (width 0) (type default) (color 0 0 0 0))
@@
     (stroke (width 0) (type default) (color 0 0 0 0))
   )
+  (wire (pts (xy 304.8 144.78) (xy 304.8 146.685))
+    (stroke (width 0) (type default) (color 0 0 0 0))
+  )
   (wire (pts (xy 258.445 156.21) (xy 254 156.21))
     (stroke (width 0) (type default) (color 0 0 0 0))
@@
     (stroke (width 0) (type default) (color 0 0 0 0))
   )
-  (wire (pts (xy 299.085 144.78) (xy 299.085 147.955))
+  (wire (pts (xy 299.085 144.78) (xy 299.085 146.685))
     (stroke (width 0) (type default) (color 0 0 0 0))
   )
@@
     (stroke (width 0) (type default) (color 0 0 0 0))
   )
+  (wire (pts (xy 304.8 133.985) (xy 304.8 137.16))
+    (stroke (width 0) (type default) (color 0 0 0 0))
+  )
   (wire (pts (xy 152.4 207.645) (xy 148.59 207.645))
     (stroke (width 0) (type default) (color 0 0 0 0))
@@
     (stroke (width 0) (type default) (color 0 0 0 0))
   )
+  (wire (pts (xy 273.685 133.985) (xy 271.145 133.985))
+    (stroke (width 0) (type default) (color 0 0 0 0))
+  )
   (wire (pts (xy 131.445 146.685) (xy 131.445 156.845))
     (stroke (width 0) (type default) (color 0 0 0 0))
@@
     (stroke (width 0) (type default) (color 0 0 0 0))
   )
+  (wire (pts (xy 299.085 146.685) (xy 299.085 147.955))
+    (stroke (width 0) (type default) (color 0 0 0 0))
+  )
   (wire (pts (xy 163.83 80.645) (xy 167.005 80.645))
     (stroke (width 0) (type default) (color 0 0 0 0))
@@
     (stroke (width 0) (type default) (color 0 0 0 0))
   )
+  (wire (pts (xy 299.085 133.985) (xy 304.8 133.985))
+    (stroke (width 0) (type default) (color 0 0 0 0))
+  )
   (wire (pts (xy 116.84 195.58) (xy 131.445 195.58))
     (stroke (width 0) (type default) (color 0 0 0 0))
@@
     (stroke (width 0) (type default) (color 0 0 0 0))
   )
+  (wire (pts (xy 271.145 133.985) (xy 271.145 135.89))
+    (stroke (width 0) (type default) (color 0 0 0 0))
+  )
   (wire (pts (xy 132.08 255.905) (xy 133.35 255.905))
     (stroke (width 0) (type default) (color 0 0 0 0))
@@
     (pin "9")
   )
+  (symbol (lib_id "Device:C") (at 304.8 140.97 0) (unit 1)
+    (in_bom yes) (on_board yes)
+    (property "Reference" "C?" (id 0) (at 310.515 139.7 0)
+      (effects (font (size 1.27 1.27)) (justify right))
+    )
+    (property "Value" "100n" (id 1) (at 307.975 142.24 0)
+      (effects (font (size 1.27 1.27)) (justify left))
+    )
+    (property "Footprint" "Capacitor_SMD:C_0805_2012Metric_Pad1.18x1.45mm_HandSolder" (id 2) (at 305.7652 144.78 0)
+      (effects (font (size 1.27 1.27)) hide)
+    )
+    (property "Datasheet" "~" (id 3) (at 304.8 140.97 0)
+      (effects (font (size 1.27 1.27)) hide)
+    )
+    (pin "1")
+    (pin "2")
+  )
   (symbol (lib_id "Isolator:VO0631T") (at 140.97 210.185 0) (mirror y) (unit 1)
     (in_bom yes) (on_board yes)
@@
     (pin "2")
   )
-  (symbol (lib_id "Device:C") (at 299.085 140.97 0) (unit 1)
+  (symbol (lib_id "Device:C") (at 299.085 140.97 0) (mirror y) (unit 1)
     (in_bom yes) (on_board yes)
-    (property "Reference" "C8" (id 0) (at 304.8 139.7 0)
+    (property "Reference" "C8" (id 0) (at 293.37 139.7 0)
       (effects (font (size 1.27 1.27)) (justify right))
     )
-    (property "Value" "100n" (id 1) (at 302.26 142.24 0)
+    (property "Value" "100n" (id 1) (at 295.91 142.24 0)
       (effects (font (size 1.27 1.27)) (justify left))
     )
-    (property "Footprint" "Capacitor_SMD:C_0805_2012Metric_Pad1.18x1.45mm_HandSolder" (id 2) (at 300.0502 144.78 0)
+    (property "Footprint" "Capacitor_SMD:C_0805_2012Metric_Pad1.18x1.45mm_HandSolder" (id 2) (at 298.1198 144.78 0)
       (effects (font (size 1.27 1.27)) hide)
     )
@@
       (reference "C14") (unit 1) (value "10u") (footprint "Capacitor_SMD:C_0805_2012Metric_Pad1.18x1.45mm_HandSolder")
     )
+    (path "/517dfd81-ae3a-4f22-a1c0-2db9a54d5e39"
+      (reference "C?") (unit 1) (value "100n") (footprint "Capacitor_SMD:C_0805_2012Metric_Pad1.18x1.45mm_HandSolder")
+    )
     (path "/f48c35ed-588e-4b54-824b-40693da77b07"
