File: solari-control.kicad_sch (KiCad schematic)
At the start: 109 parts, among them J1 Conn_01x04, J2 A5081WV-5P, J3 A5081WR-5P, J4 AVR-ISP-6, J5 DIL8, J6 Conn_01x04, Q1 AO3401A, Q10 AO3400A, Q11 AO3401A, Q12 AO3400A, Q2 AO3400A, Q3 AO3401A, Q4 AO3400A, Q5 AO3401A, Q6 AO3401A, Q7 AO3401A, Q8 AO3401A, Q9 AO3401A, U1 VO0631T, U10 PC817, U11 PC817, U12 AMS1117-3.3, U2 L78L05_SOT89, U3 VO0631T, U4 PC817, U5 PC817, U6 VO0631T, U7 ATmega328P-A, U8 VO0631T, U9 VO0631T, Y1 14.7456 MHz

Commit message: PCB: partially wire galvanic separation on IO.
Parts:
- gave numbers to parts that had none: 1
Connections:
- net 0PH: now also C5.2, Q2.2 (S), Q4.2 (S), R12.1, R9.1, U3.5 (GND)
- net VPH: no longer C5.2, Q2.2 (S), Q4.2 (S), R12.1, R9.1, U3.5 (GND)
Changed lines of the file:
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@@
     )
   )
-  (global_label "VPH" (shape input) (at 74.295 90.805 180) (fields_autoplaced)
+  (global_label "0PH" (shape input) (at 74.295 90.805 180) (fields_autoplaced)
     (effects (font (size 1.27 1.27)) (justify right))
-    (property "Intersheet References" "${INTERSHEET_REFS}" (id 0) (at 68.1929 90.8844 0)
+    (property "Intersheet References" "${INTERSHEET_REFS}" (id 0) (at 68.0719 90.7256 0)
       (effects (font (size 1.27 1.27)) (justify right) hide)
     )
@@
   (symbol (lib_id "Device:C") (at 304.8 140.97 0) (unit 1)
     (in_bom yes) (on_board yes)
-    (property "Reference" "C?" (id 0) (at 310.515 139.7 0)
-      (effects (font (size 1.27 1.27)) (justify right))
+    (property "Reference" "C15" (id 0) (at 307.975 139.7 0)
+      (effects (font (size 1.27 1.27)) (justify left))
     )
     (property "Value" "100n" (id 1) (at 307.975 142.24 0)
@@
     )
     (path "/517dfd81-ae3a-4f22-a1c0-2db9a54d5e39"
-      (reference "C?") (unit 1) (value "100n") (footprint "Capacitor_SMD:C_0805_2012Metric_Pad1.18x1.45mm_HandSolder")
+      (reference "C15") (unit 1) (value "100n") (footprint "Capacitor_SMD:C_0805_2012Metric_Pad1.18x1.45mm_HandSolder")
     )
     (path "/f48c35ed-588e-4b54-824b-40693da77b07"

Commit message: Wire whole PCB.
Parts:
- U2: footprint Package_TO_SOT_SMD:SOT-89-3 -> Package_TO_SOT_SMD:SOT-89-3_Handsoldering
Connections:
- net TX: now also D1.4 (IO3); no longer D1.5 (IO4)
- net V+: no longer F3.1, J3.3 (Pin_3)
- net VDO: no longer F4.1, J3.5 (Pin_5)
- net VPH: no longer F2.1, J2.4 (Pin_4)
- new net _V+: F3.1, J3.3 (Pin_3)
- new net _VDO: F4.1, J3.5 (Pin_5)
- new net _VPH: F2.1, J2.4 (Pin_4)
Changed lines of the file:
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@@
   (junction (at 108.585 195.58) (diameter 0) (color 0 0 0 0)
   )
-  (junction (at 356.235 47.625) (diameter 0) (color 0 0 0 0)
-  )
   (junction (at 152.4 212.725) (diameter 0) (color 0 0 0 0)
   )
@@
   (junction (at 265.43 30.48) (diameter 0) (color 0 0 0 0)
   )
+  (junction (at 353.695 47.625) (diameter 0) (color 0 0 0 0)
+  )
   (junction (at 119.38 215.265) (diameter 0) (color 0 0 0 0)
   )
@@
   (no_connect (at 288.925 151.13))
   (no_connect (at 148.59 184.15))
-  (no_connect (at 353.695 50.8))
+  (no_connect (at 356.235 50.8))
   (no_connect (at 288.925 148.59))
   (no_connect (at 258.445 148.59))
@@
     (stroke (width 0) (type default) (color 0 0 0 0))
   )
-  (wire (pts (xy 334.645 47.625) (xy 356.235 47.625))
+  (wire (pts (xy 334.645 47.625) (xy 353.695 47.625))
     (stroke (width 0) (type default) (color 0 0 0 0))
   )
@@
     (stroke (width 0) (type default) (color 0 0 0 0))
   )
-  (wire (pts (xy 356.235 47.625) (xy 371.475 47.625))
+  (wire (pts (xy 353.695 47.625) (xy 371.475 47.625))
     (stroke (width 0) (type default) (color 0 0 0 0))
   )
@@
     (stroke (width 0) (type default) (color 0 0 0 0))
   )
-  (wire (pts (xy 356.235 47.625) (xy 356.235 50.8))
+  (wire (pts (xy 353.695 47.625) (xy 353.695 50.8))
     (stroke (width 0) (type default) (color 0 0 0 0))
   )
@@
     (effects (font (size 1.27 1.27)) (justify left bottom))
   )
-  (label "VPH" (at 239.395 49.53 0)
+  (label "_VPH" (at 239.395 49.53 0)
     (effects (font (size 1.27 1.27)) (justify left bottom))
   )
@@
     (effects (font (size 1.27 1.27)) (justify left bottom))
   )
-  (label "V+" (at 239.395 86.36 0)
+  (label "_V+" (at 239.395 86.36 0)
     (effects (font (size 1.27 1.27)) (justify left bottom))
   )
-  (label "VDO" (at 239.395 91.44 0)
+  (label "_VDO" (at 239.395 91.44 0)
     (effects (font (size 1.27 1.27)) (justify left bottom))
   )
@@
     (property "Reference" "U2" (id 0) (at 284.48 47.1002 0))
     (property "Value" "L78L05_SOT89" (id 1) (at 284.48 49.6371 0))
-    (property "Footprint" "Package_TO_SOT_SMD:SOT-89-3" (id 2) (at 284.48 47.625 0)
+    (property "Footprint" "Package_TO_SOT_SMD:SOT-89-3_Handsoldering" (id 2) (at 284.48 47.625 0)
       (effects (font (size 1.27 1.27) italic) hide)
     )
@@
     )
     (path "/1a16ae63-bc3a-42bf-b35a-01e42f7e525a"
-      (reference "U2") (unit 1) (value "L78L05_SOT89") (footprint "Package_TO_SOT_SMD:SOT-89-3")
+      (reference "U2") (unit 1) (value "L78L05_SOT89") (footprint "Package_TO_SOT_SMD:SOT-89-3_Handsoldering")
     )
     (path "/5f201b59-27c5-4aad-9141-a0b47a4ce738"

Commit message: Add test points for remaining grounds.
Parts:
- added TP2, TP3: TP, TestPoint:TestPoint_Loop_D3.50mm_Drill1.4mm_Beaded, symbol Connector:TestPoint
Connections:
- net 0PH: now also TP3.1
- net 0V+: now also TP2.1
Other:
- moved on the sheet: H1, H2, H3, H4, TP1
Changed lines of the file:
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@@
     (stroke (width 0) (type default) (color 0 0 0 0))
   )
+  (wire (pts (xy 261.62 269.875) (xy 261.62 272.415))
+    (stroke (width 0) (type default) (color 0 0 0 0))
+  )
   (wire (pts (xy 97.155 210.185) (xy 108.585 210.185))
     (stroke (width 0) (type default) (color 0 0 0 0))
@@
     (stroke (width 0) (type default) (color 0 0 0 0))
   )
+  (wire (pts (xy 252.095 269.875) (xy 252.095 272.415))
+    (stroke (width 0) (type default) (color 0 0 0 0))
+  )
   (wire (pts (xy 131.445 128.27) (xy 125.095 128.27))
     (stroke (width 0) (type default) (color 0 0 0 0))
@@
     )
   )
+  (global_label "0V+" (shape input) (at 252.095 272.415 270) (fields_autoplaced)
+    (effects (font (size 1.27 1.27)) (justify right))
+    (property "Intersheet References" "${INTERSHEET_REFS}" (id 0) (at 252.1744 278.6986 90)
+      (effects (font (size 1.27 1.27)) (justify right) hide)
+    )
+  )
   (global_label "MP" (shape input) (at 167.005 111.76 0) (fields_autoplaced)
     (effects (font (size 1.27 1.27)) (justify left))
@@
     )
   )
+  (global_label "0PH" (shape input) (at 261.62 272.415 270) (fields_autoplaced)
+    (effects (font (size 1.27 1.27)) (justify right))
+    (property "Intersheet References" "${INTERSHEET_REFS}" (id 0) (at 261.6994 278.6381 90)
+      (effects (font (size 1.27 1.27)) (justify right) hide)
+    )
+  )
   (global_label "MISO" (shape input) (at 254 153.67 180) (fields_autoplaced)
     (effects (font (size 1.27 1.27)) (justify right))
@@
     (pin "2")
   )
+  (symbol (lib_id "Connector:TestPoint") (at 252.095 269.875 0) (unit 1)
+    (in_bom yes) (on_board yes) (fields_autoplaced)
+    (property "Reference" "TP2" (id 0) (at 253.492 265.7383 0)
+      (effects (font (size 1.27 1.27)) (justify left))
+    )
+    (property "Value" "TP" (id 1) (at 253.492 268.2752 0)
+      (effects (font (size 1.27 1.27)) (justify left))
+    )
+    (property "Footprint" "TestPoint:TestPoint_Loop_D3.50mm_Drill1.4mm_Beaded" (id 2) (at 257.175 269.875 0)
+      (effects (font (size 1.27 1.27)) hide)
+    )
+    (property "Datasheet" "~" (id 3) (at 257.175 269.875 0)
+      (effects (font (size 1.27 1.27)) hide)
+    )
+    (pin "1")
+  )
   (symbol (lib_id "Connector_Generic:Conn_01x05") (at 233.68 86.36 0) (mirror y) (unit 1)
     (in_bom yes) (on_board yes) (fields_autoplaced)
@@
     (pin "3")
   )
+  (symbol (lib_id "Connector:TestPoint") (at 261.62 269.875 0) (unit 1)
+    (in_bom yes) (on_board yes) (fields_autoplaced)
+    (property "Reference" "TP3" (id 0) (at 263.017 265.7383 0)
+      (effects (font (size 1.27 1.27)) (justify left))
+    )
+    (property "Value" "TP" (id 1) (at 263.017 268.2752 0)
+      (effects (font (size 1.27 1.27)) (justify left))
+    )
+    (property "Footprint" "TestPoint:TestPoint_Loop_D3.50mm_Drill1.4mm_Beaded" (id 2) (at 266.7 269.875 0)
+      (effects (font (size 1.27 1.27)) hide)
+    )
+    (property "Datasheet" "~" (id 3) (at 266.7 269.875 0)
+      (effects (font (size 1.27 1.27)) hide)
+    )
+    (pin "1")
+  )
   (symbol (lib_id "Device:C") (at 262.255 85.09 0) (mirror y) (unit 1)
     (in_bom yes) (on_board yes)
@@
     (pin "8")
   )
-  (symbol (lib_id "Mechanical:MountingHole") (at 252.73 273.05 0) (mirror y) (unit 1)
+  (symbol (lib_id "Mechanical:MountingHole") (at 231.14 273.05 0) (mirror y) (unit 1)
     (in_bom yes) (on_board yes)
-    (property "Reference" "H3" (id 0) (at 250.19 272.415 0)
+    (property "Reference" "H3" (id 0) (at 228.6 272.415 0)
       (effects (font (size 1.27 1.27)) (justify left))
     )
-    (property "Value" "MH" (id 1) (at 250.19 274.32 0)
+    (property "Value" "MH" (id 1) (at 228.6 274.32 0)
       (effects (font (size 1.27 1.27)) (justify left))
     )
-    (property "Footprint" "MountingHole:MountingHole_3mm_Pad_Via" (id 2) (at 252.73 273.05 0)
+    (property "Footprint" "MountingHole:MountingHole_3mm_Pad_Via" (id 2) (at 231.14 273.05 0)
       (effects (font (size 1.27 1.27)) hide)
     )
-    (property "Datasheet" "~" (id 3) (at 252.73 273.05 0)
+    (property "Datasheet" "~" (id 3) (at 231.14 273.05 0)
       (effects (font (size 1.27 1.27)) hide)
     )
@@
     (pin "2")
   )
-  (symbol (lib_id "Mechanical:MountingHole") (at 252.73 266.7 0) (unit 1)
+  (symbol (lib_id "Mechanical:MountingHole") (at 231.14 266.7 0) (unit 1)
     (in_bom yes) (on_board yes)
-    (property "Reference" "H1" (id 0) (at 250.19 266.065 0)
+    (property "Reference" "H1" (id 0) (at 228.6 266.065 0)
       (effects (font (size 1.27 1.27)) (justify right))
     )
-    (property "Value" "MH" (id 1) (at 250.19 267.97 0)
+    (property "Value" "MH" (id 1) (at 228.6 267.97 0)
       (effects (font (size 1.27 1.27)) (justify right))
     )
-    (property "Footprint" "MountingHole:MountingHole_3mm_Pad_Via" (id 2) (at 252.73 266.7 0)
+    (property "Footprint" "MountingHole:MountingHole_3mm_Pad_Via" (id 2) (at 231.14 266.7 0)
       (effects (font (size 1.27 1.27)) hide)
     )
-    (property "Datasheet" "~" (id 3) (at 252.73 266.7 0)
+    (property "Datasheet" "~" (id 3) (at 231.14 266.7 0)
       (effects (font (size 1.27 1.27)) hide)
     )
@@
     (pin "2")
   )
-  (symbol (lib_id "Mechanical:MountingHole") (at 259.08 266.7 0) (unit 1)
+  (symbol (lib_id "Mechanical:MountingHole") (at 237.49 266.7 0) (unit 1)
     (in_bom yes) (on_board yes) (fields_autoplaced)
-    (property "Reference" "H2" (id 0) (at 261.62 265.8653 0)
+    (property "Reference" "H2" (id 0) (at 240.03 265.8653 0)
       (effects (font (size 1.27 1.27)) (justify left))
     )
-    (property "Value" "MH" (id 1) (at 261.62 268.4022 0)
+    (property "Value" "MH" (id 1) (at 240.03 268.4022 0)
       (effects (font (size 1.27 1.27)) (justify left))
     )
-    (property "Footprint" "MountingHole:MountingHole_3mm_Pad_Via" (id 2) (at 259.08 266.7 0)
+    (property "Footprint" "MountingHole:MountingHole_3mm_Pad_Via" (id 2) (at 237.49 266.7 0)
       (effects (font (size 1.27 1.27)) hide)
     )
-    (property "Datasheet" "~" (id 3) (at 259.08 266.7 0)
+    (property "Datasheet" "~" (id 3) (at 237.49 266.7 0)
       (effects (font (size 1.27 1.27)) hide)
     )
@@
     (pin "3")
   )
-  (symbol (lib_id "Connector:TestPoint") (at 273.05 269.875 0) (unit 1)
+  (symbol (lib_id "Connector:TestPoint") (at 271.145 269.875 0) (unit 1)
     (in_bom yes) (on_board yes) (fields_autoplaced)
-    (property "Reference" "TP1" (id 0) (at 274.447 265.7383 0)
+    (property "Reference" "TP1" (id 0) (at 272.542 265.7383 0)
       (effects (font (size 1.27 1.27)) (justify left))
     )
-    (property "Value" "TP" (id 1) (at 274.447 268.2752 0)
+    (property "Value" "TP" (id 1) (at 272.542 268.2752 0)
       (effects (font (size 1.27 1.27)) (justify left))
     )
-    (property "Footprint" "TestPoint:TestPoint_Loop_D3.50mm_Drill1.4mm_Beaded" (id 2) (at 278.13 269.875 0)
+    (property "Footprint" "TestPoint:TestPoint_Loop_D3.50mm_Drill1.4mm_Beaded" (id 2) (at 276.225 269.875 0)
       (effects (font (size 1.27 1.27)) hide)
     )
-    (property "Datasheet" "~" (id 3) (at 278.13 269.875 0)
+    (property "Datasheet" "~" (id 3) (at 276.225 269.875 0)
       (effects (font (size 1.27 1.27)) hide)
     )
@@
     (pin "5")
   )
-  (symbol (lib_id "power:GND") (at 273.05 269.875 0) (unit 1)
+  (symbol (lib_id "power:GND") (at 271.145 269.875 0) (unit 1)
     (in_bom yes) (on_board yes) (fields_autoplaced)
-    (property "Reference" "#PWR018" (id 0) (at 273.05 276.225 0)
+    (property "Reference" "#PWR018" (id 0) (at 271.145 276.225 0)
       (effects (font (size 1.27 1.27)) hide)
     )
-    (property "Value" "GND" (id 1) (at 273.05 274.3184 0))
-    (property "Footprint" "" (id 2) (at 273.05 269.875 0)
+    (property "Value" "GND" (id 1) (at 271.145 274.3184 0))
+    (property "Footprint" "" (id 2) (at 271.145 269.875 0)
       (effects (font (size 1.27 1.27)) hide)
     )
-    (property "Datasheet" "" (id 3) (at 273.05 269.875 0)
+    (property "Datasheet" "" (id 3) (at 271.145 269.875 0)
       (effects (font (size 1.27 1.27)) hide)
     )
@@
     (pin "2")
   )
-  (symbol (lib_id "Mechanical:MountingHole") (at 259.08 273.05 0) (unit 1)
+  (symbol (lib_id "Mechanical:MountingHole") (at 237.49 273.05 0) (unit 1)
     (in_bom yes) (on_board yes) (fields_autoplaced)
-    (property "Reference" "H4" (id 0) (at 261.62 272.2153 0)
+    (property "Reference" "H4" (id 0) (at 240.03 272.2153 0)
       (effects (font (size 1.27 1.27)) (justify left))
     )
-    (property "Value" "MH" (id 1) (at 261.62 274.7522 0)
+    (property "Value" "MH" (id 1) (at 240.03 274.7522 0)
       (effects (font (size 1.27 1.27)) (justify left))
     )
-    (property "Footprint" "MountingHole:MountingHole_3mm_Pad_Via" (id 2) (at 259.08 273.05 0)
+    (property "Footprint" "MountingHole:MountingHole_3mm_Pad_Via" (id 2) (at 237.49 273.05 0)
       (effects (font (size 1.27 1.27)) hide)
     )
-    (property "Datasheet" "~" (id 3) (at 259.08 273.05 0)
+    (property "Datasheet" "~" (id 3) (at 237.49 273.05 0)
       (effects (font (size 1.27 1.27)) hide)
     )
@@
       (reference "TP1") (unit 1) (value "TP") (footprint "TestPoint:TestPoint_Loop_D3.50mm_Drill1.4mm_Beaded")
     )
+    (path "/03d49c74-a211-4fbc-bc38-560cb47f3670"
+      (reference "TP2") (unit 1) (value "TP") (footprint "TestPoint:TestPoint_Loop_D3.50mm_Drill1.4mm_Beaded")
+    )
+    (path "/49de7fa4-491f-405e-ad2d-91b69b77b0a6"
+      (reference "TP3") (unit 1) (value "TP") (footprint "TestPoint:TestPoint_Loop_D3.50mm_Drill1.4mm_Beaded")
+    )
     (path "/9189084f-e9e7-4600-82e7-b2d1b5370df8"

Commit message: Sch: use galvanic separation on UART interface.
Parts:
- removed JP1: J2O, Connector_PinHeader_2.54mm:PinHeader_1x02_P2.54mm_Vertical, symbol Jumper:Jumper_2_Open
- added C16, C17: 100n, Capacitor_SMD:C_0805_2012Metric_Pad1.18x1.45mm_HandSolder, symbol Device:C
- added U13: ADuM1201AR, Package_SO:SOIC-8_3.9x4.9mm_P1.27mm, symbol Isolator:ADuM1201AR
Connections:
- net GND: now also C16.2, U13.4 (GND1); no longer D1.2 (GND), J1.4 (Pin_4)
- net RX: now also U13.2 (VOA); no longer D1.6 (IO5), J1.2 (Pin_2)
- net TX: now also U13.3 (VIB); no longer D1.4 (IO3), J1.3 (Pin_3)
- net VCC: now also C16.1, U13.1 (VDD1)
- net VCCU: now reaches J1.1 (Pin_1)
- net VCCU: now also C17.1, U13.8 (VDD2)
- new net GNDU: C17.2, D1.2 (GND), J1.4 (Pin_4), U13.5 (GND2)
- new net RXU: D1.6 (IO5), J1.2 (Pin_2), U13.7 (VIA)
- new net TXU: D1.4 (IO3), J1.3 (Pin_3), U13.6 (VOB)
Other:
- note added: "Galvanically separated"
- moved on the sheet: D1, D4, D5, D6, J1, R26, R27, R28

Commit message: Sch: power logic from 5V.
Parts:
- removed C14: 10u, Capacitor_SMD:C_0805_2012Metric_Pad1.18x1.45mm_HandSolder, symbol Device:C
- removed JP2: Jumper_3_Open, Connector_PinHeader_2.54mm:PinHeader_1x03_P2.54mm_Vertical, symbol Jumper:Jumper_3_Open
- removed U12: AMS1117-3.3, Package_TO_SOT_SMD:SOT-223-3_TabPin2, symbol Regulator_Linear:AMS1117-3.3
- added JP1: Jumper_2_Open, Connector_PinHeader_2.54mm:PinHeader_1x02_P2.54mm_Vertical, symbol Jumper:Jumper_2_Open
- C2: value 22u/25V -> 22u
Connections:
- net VCC: now also C2.1, F1.2, JP1.1 (A)
- net at J4.2 (VCC): now also JP1.2 (B)
Other:
- note removed: "Parent device has 3.3V UART."
- moved on the sheet: H1, H2, H3, H4, TP2, TP3

Commit message: Wire new changes on PCB.
Changed lines of the file:
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@@
   (junction (at 151.13 49.53) (diameter 0) (color 0 0 0 0)
   )
+  (junction (at 360.045 185.42) (diameter 0) (color 0 0 0 0)
+  )
   (junction (at 96.52 273.685) (diameter 0) (color 0 0 0 0)
   )
@@
   (junction (at 152.4 145.415) (diameter 0) (color 0 0 0 0)
   )
-  (junction (at 245.11 96.52) (diameter 0) (color 0 0 0 0)
-  )
   (junction (at 262.255 96.52) (diameter 0) (color 0 0 0 0)
   )
@@
   (junction (at 152.4 207.645) (diameter 0) (color 0 0 0 0)
   )
-  (junction (at 245.11 81.28) (diameter 0) (color 0 0 0 0)
-  )
   (junction (at 93.345 251.46) (diameter 0) (color 0 0 0 0)
   )
@@
   (junction (at 131.445 195.58) (diameter 0) (color 0 0 0 0)
   )
+  (junction (at 365.125 197.485) (diameter 0) (color 0 0 0 0)
+  )
   (junction (at 217.805 163.83) (diameter 0) (color 0 0 0 0)
   )
   (junction (at 282.956 88.9) (diameter 0) (color 0 0 0 0)
   )
-  (junction (at 245.11 52.705) (diameter 0) (color 0 0 0 0)
-  )
   (junction (at 125.095 161.925) (diameter 0) (color 0 0 0 0)
   )
@@
     (stroke (width 0) (type default) (color 0 0 0 0))
   )
-  (wire (pts (xy 365.125 193.04) (xy 365.125 210.185))
+  (wire (pts (xy 365.125 193.04) (xy 365.125 197.485))
     (stroke (width 0) (type default) (color 0 0 0 0))
   )
@@
     (stroke (width 0) (type default) (color 0 0 0 0))
   )
-  (wire (pts (xy 345.44 185.42) (xy 372.11 185.42))
+  (wire (pts (xy 345.44 185.42) (xy 360.045 185.42))
     (stroke (width 0) (type default) (color 0 0 0 0))
   )
@@
     (stroke (width 0) (type default) (color 0 0 0 0))
   )
+  (wire (pts (xy 360.045 185.42) (xy 372.11 185.42))
+    (stroke (width 0) (type default) (color 0 0 0 0))
+  )
   (wire (pts (xy 299.085 133.985) (xy 304.8 133.985))
     (stroke (width 0) (type default) (color 0 0 0 0))
@@
     (stroke (width 0) (type default) (color 0 0 0 0))
   )
+  (wire (pts (xy 365.125 197.485) (xy 365.125 210.185))
+    (stroke (width 0) (type default) (color 0 0 0 0))
+  )
   (wire (pts (xy 238.76 91.44) (xy 245.11 91.44))
     (stroke (width 0) (type default) (color 0 0 0 0))
@@
     (pin "2")
   )
-  (symbol (lib_id "power:PWR_FLAG") (at 245.11 52.705 180) (unit 1)
+  (symbol (lib_id "power:PWR_FLAG") (at 262.255 52.705 0) (unit 1)
     (in_bom yes) (on_board yes)
-    (property "Reference" "#FLG03" (id 0) (at 245.11 54.61 0)
+    (property "Reference" "#FLG03" (id 0) (at 262.255 50.8 0)
       (effects (font (size 1.27 1.27)) hide)
     )
-    (property "Value" "PWR_FLAG" (id 1) (at 243.84 56.515 0))
-    (property "Footprint" "" (id 2) (at 245.11 52.705 0)
+    (property "Value" "PWR_FLAG" (id 1) (at 263.525 48.895 0))
+    (property "Footprint" "" (id 2) (at 262.255 52.705 0)
       (effects (font (size 1.27 1.27)) hide)
     )
-    (property "Datasheet" "~" (id 3) (at 245.11 52.705 0)
+    (property "Datasheet" "~" (id 3) (at 262.255 52.705 0)
       (effects (font (size 1.27 1.27)) hide)
     )
@@
     (pin "3")
   )
-  (symbol (lib_id "power:PWR_FLAG") (at 245.11 96.52 180) (unit 1)
+  (symbol (lib_id "power:PWR_FLAG") (at 262.255 96.52 180) (unit 1)
     (in_bom yes) (on_board yes) (fields_autoplaced)
-    (property "Reference" "#FLG07" (id 0) (at 245.11 98.425 0)
+    (property "Reference" "#FLG07" (id 0) (at 262.255 98.425 0)
       (effects (font (size 1.27 1.27)) hide)
     )
-    (property "Value" "PWR_FLAG" (id 1) (at 245.11 100.9634 0))
-    (property "Footprint" "" (id 2) (at 245.11 96.52 0)
+    (property "Value" "PWR_FLAG" (id 1) (at 262.255 100.9634 0))
+    (property "Footprint" "" (id 2) (at 262.255 96.52 0)
       (effects (font (size 1.27 1.27)) hide)
     )
-    (property "Datasheet" "~" (id 3) (at 245.11 96.52 0)
+    (property "Datasheet" "~" (id 3) (at 262.255 96.52 0)
       (effects (font (size 1.27 1.27)) hide)
     )
@@
     (pin "2")
   )
-  (symbol (lib_id "power:PWR_FLAG") (at 245.11 81.28 0) (unit 1)
+  (symbol (lib_id "power:PWR_FLAG") (at 262.255 81.28 0) (unit 1)
     (in_bom yes) (on_board yes) (fields_autoplaced)
-    (property "Reference" "#FLG05" (id 0) (at 245.11 79.375 0)
+    (property "Reference" "#FLG05" (id 0) (at 262.255 79.375 0)
       (effects (font (size 1.27 1.27)) hide)
     )
-    (property "Value" "PWR_FLAG" (id 1) (at 245.11 77.7042 0))
-    (property "Footprint" "" (id 2) (at 245.11 81.28 0)
+    (property "Value" "PWR_FLAG" (id 1) (at 262.255 77.7042 0))
+    (property "Footprint" "" (id 2) (at 262.255 81.28 0)
       (effects (font (size 1.27 1.27)) hide)
     )
-    (property "Datasheet" "~" (id 3) (at 245.11 81.28 0)
+    (property "Datasheet" "~" (id 3) (at 262.255 81.28 0)
       (effects (font (size 1.27 1.27)) hide)
     )
@@
     (pin "4")
   )
+  (symbol (lib_id "power:PWR_FLAG") (at 360.045 185.42 0) (unit 1)
+    (in_bom yes) (on_board yes) (fields_autoplaced)
+    (property "Reference" "#FLG0101" (id 0) (at 360.045 183.515 0)
+      (effects (font (size 1.27 1.27)) hide)
+    )
+    (property "Value" "PWR_FLAG" (id 1) (at 360.045 181.8442 0))
+    (property "Footprint" "" (id 2) (at 360.045 185.42 0)
+      (effects (font (size 1.27 1.27)) hide)
+    )
+    (property "Datasheet" "~" (id 3) (at 360.045 185.42 0)
+      (effects (font (size 1.27 1.27)) hide)
+    )
+    (pin "1")
+  )
   (symbol (lib_id "Device:C") (at 131.445 73.025 0) (mirror y) (unit 1)
     (in_bom yes) (on_board yes)
@@
     (pin "2")
   )
+  (symbol (lib_id "power:PWR_FLAG") (at 365.125 197.485 270) (unit 1)
+    (in_bom yes) (on_board yes) (fields_autoplaced)
+    (property "Reference" "#FLG08" (id 0) (at 367.03 197.485 0)
+      (effects (font (size 1.27 1.27)) hide)
+    )
+    (property "Value" "PWR_FLAG" (id 1) (at 368.3 197.9188 90)
+      (effects (font (size 1.27 1.27)) (justify left))
+    )
+    (property "Footprint" "" (id 2) (at 365.125 197.485 0)
+      (effects (font (size 1.27 1.27)) hide)
+    )
+    (property "Datasheet" "~" (id 3) (at 365.125 197.485 0)
+      (effects (font (size 1.27 1.27)) hide)
+    )
+    (pin "1")
+  )
   (symbol (lib_id "Device:R") (at 125.095 205.105 90) (unit 1)
     (in_bom yes) (on_board yes) (fields_autoplaced)
@@
       (reference "#FLG07") (unit 1) (value "PWR_FLAG") (footprint "")
     )
+    (path "/e580202e-9730-4152-a8cd-7555450a6e7e"
+      (reference "#FLG08") (unit 1) (value "PWR_FLAG") (footprint "")
+    )
+    (path "/e06e06f2-1667-42cc-a194-df3c1c432a44"
+      (reference "#FLG0101") (unit 1) (value "PWR_FLAG") (footprint "")
+    )
     (path "/1b547ee9-4e83-4450-a053-2e5e57da3d6a"
