File: solari-control.kicad_pcb (KiCad board)
At the start: 2 copper layers, 80 x 80 mm, 108 parts, among them J1 Conn_01x04, J2 A5081WV-5P, J3 A5081WR-5P, J4 AVR-ISP-6, J5 DIL8, J6 Conn_01x04, Q1 AO3401A, Q10 AO3400A, Q11 AO3401A, Q12 AO3400A, Q2 AO3400A, Q3 AO3401A, Q4 AO3400A, Q5 AO3401A, Q6 AO3401A, Q7 AO3401A, Q8 AO3401A, Q9 AO3401A, U1 VO0631T, U10 PC817, U11 PC817, U2 L78L05_SOT89, U3 VO0631T, U4 PC817, U5 PC817, U6 VO0631T, U7 ATmega328P-A, U8 VO0631T, U9 VO0631T, Y1 14.7456 MHz

Commit message: PCB: place parts into chunks.
Parts:
- removed C14: 22u/25V, Capacitor_SMD:C_0805_2012Metric_Pad1.18x1.45mm_HandSolder
- removed C15: 100n, Capacitor_SMD:C_0805_2012Metric_Pad1.18x1.45mm_HandSolder
- D5, D6, Q11, Q12, R41, R42, R43, R44, R45, R46, U10, U11: moved to B.Cu
- moved R27 152.6 mm to (229.1, 90.4), turned to -90 degrees
- moved R28 146.2 mm to (232.7, 90.4), turned to -90 degrees
- moved D6 139.7 mm to (232.2, 85.6), turned to -90 degrees
- moved D4 129.3 mm to (225.6, 85.3), turned to -90 degrees
- moved R29 126.5 mm to (174.5, 23.4)
- moved R22 123.5 mm to (190.2, 22.9)
- moved D5 121.1 mm to (228.9, 85.3), turned to -90 degrees
- moved R23 118.2 mm to (192.8, 33.5)
- moved C9 117.1 mm to (195.3, 29.0), turned to -90 degrees
- moved R31 111.4 mm to (150.6, 21.3)
- moved R1 110.8 mm to (180.3, 71.6)
- moved R34 109.9 mm to (155.2, 21.1)
- moved R25 109.3 mm to (188.7, 33.5)
- moved D1 107.5 mm to (209.8, 92.2)
- moved R33 105.9 mm to (150.9, 23.9)
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Connections:
- R42 pad 1: VDO -> Net-(Q11-Pad1)
- R42 pad 2: Net-(Q11-Pad1) -> VDO

Commit message: Use 3V3 power supply.
Parts:
- added C14: 10u, Capacitor_SMD:C_0805_2012Metric_Pad1.18x1.45mm_HandSolder, F.Cu at (131.7, 85.0)
- added U12: AMS1117-3.3, Package_TO_SOT_SMD:SOT-223-3_TabPin2, F.Cu at (124.4, 87.6)
Connections:
- C2 pad 1: VCC -> Net-(C2-Pad1)
- F1 pad 1: VCC -> Net-(F1-Pad1)
- F1 pad 2: VCC -> Net-(C2-Pad1)
- J2 pad 1: VCC -> Net-(F1-Pad1)

Commit message: Add power jumper for AVR-ISP connector.
Parts:
- JP2: value SJ2O -> Jumper_3_Open; footprint Jumper:SolderJumper-2_P1.3mm_Open_RoundedPad1.0x1.5mm -> Connector_PinHeader_2.54mm:PinHeader_1x03_P2.54mm_Vertical
- moved JP2 85.8 mm to (124.3, 73.8)
Connections:
- F1 pad 1: Net-(F1-Pad1) -> 5V
- J2 pad 1: Net-(F1-Pad1) -> 5V
- JP2 pad 1: Net-(J4-Pad2) -> VCC
- JP2 pad 2: VCC -> Net-(J4-Pad2)

Commit message: PCB: partially wire galvanic separation on IO.
Parts:
- added C15: 100n, Capacitor_SMD:C_0805_2012Metric_Pad1.18x1.45mm_HandSolder, B.Cu at (186.2, 105.3)
- C14, U12: moved to B.Cu
- moved C13 58.4 mm to (188.0, 80.2)
- moved R31 56.0 mm to (185.9, 64.8)
- moved R33 55.6 mm to (185.9, 67.0)
- moved R36 53.9 mm to (185.9, 58.1)
- moved Q7 53.8 mm to (185.9, 61.5)
- moved R38 53.8 mm to (181.6, 58.1)
- moved Q8 53.6 mm to (181.6, 61.5)
- moved R37 53.2 mm to (184.2, 81.8)
- moved U9 53.2 mm to (184.9, 73.4), turned to 90 degrees
- moved R32 53.2 mm to (184.7, 79.2)
- moved R5 52.4 mm to (222.8, 69.6)
- moved R11 52.4 mm to (232.4, 68.6)
- moved R34 51.0 mm to (181.6, 64.8), turned to 0 degrees
- moved R35 50.6 mm to (181.6, 67.0)
- moved R23 48.4 mm to (180.1, 80.2), turned to -90 degrees
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Connections:
- C5 pad 2: VPH -> 0PH
- Q2 pad 2: VPH -> 0PH
- Q4 pad 2: VPH -> 0PH
- R12 pad 1: VPH -> 0PH
- R9 pad 1: VPH -> 0PH
- U3 pad 5: VPH -> 0PH
- U7 pad 18: unconnected-(U7-Pad18) -> VCC
Routing:
- net /REL1: track 0.00 -> 9.46 mm
- net /REL2: track 0.00 -> 9.45 mm
- net Net-(R35-Pad2): track 0.00 -> 6.73 mm
- net Net-(R6-Pad2): track 0.00 -> 5.69 mm
- net Net-(R10-Pad2): track 0.00 -> 5.46 mm
- net Net-(Q11-Pad3): track 0.00 -> 5.18 mm
- net Net-(Q10-Pad1): track 0.00 -> 5.16 mm
- net Net-(Q1-Pad3): track 0.00 -> 5.16 mm
- net Net-(Q3-Pad3): track 0.00 -> 5.16 mm
- net Net-(R44-Pad2): track 0.00 -> 5.13 mm
- net Net-(R40-Pad2): track 0.00 -> 5.13 mm
- net /Z: track 0.00 -> 5.09 mm
- net /P: track 0.00 -> 5.09 mm
- net Net-(R14-Pad2): track 0.00 -> 4.82 mm
- net VPH: track 0.00 -> 4.78 mm
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- added copper zone on B.Cu, net 0PH
- added copper zone on B.Cu, net 0V+

Commit message: Wire whole PCB.
Parts:
- C3, C4, C6, C7, D4, D5, D6, F2, F3, F4, R26, R27, R28: moved to F.Cu
- U2: footprint Package_TO_SOT_SMD:SOT-89-3 -> Package_TO_SOT_SMD:SOT-89-3_Handsoldering; moved to F.Cu
- moved R11 84.9 mm to (148.3, 80.3), turned to -90 degrees
- moved D6 82.6 mm to (149.6, 87.6), turned to 0 degrees
- moved D5 79.4 mm to (149.6, 90.2), turned to 0 degrees
- moved R28 78.5 mm to (154.2, 87.6), turned to 180 degrees
- moved D4 76.3 mm to (149.6, 92.7), turned to 0 degrees
- moved R27 74.9 mm to (154.2, 90.2), turned to 180 degrees
- moved R5 72.7 mm to (150.9, 80.3), turned to -90 degrees
- moved R26 71.4 mm to (154.2, 92.7), turned to 180 degrees
- moved F4 63.3 mm to (217.2, 116.4), turned to 90 degrees
- moved C7 52.4 mm to (216.2, 109.5), turned to 0 degrees
- moved JP2 48.8 mm to (158.8, 108.5), turned to 180 degrees
- moved C3 42.5 mm to (145.8, 114.8), turned to 0 degrees
- moved C10 39.5 mm to (195.4, 107.2), turned to -90 degrees
- moved Y1 38.2 mm to (190.7, 103.4)
- moved C6 31.7 mm to (213.4, 112.3), turned to 0 degrees
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Connections:
- D1 pad 4: unconnected-(D1-Pad4) -> TX
- D1 pad 5: TX -> unconnected-(D1-Pad5)
- F2 pad 1: VPH -> /_VPH
- F3 pad 1: V+ -> /_V+
- F4 pad 1: VDO -> /_VDO
- J2 pad 4: VPH -> /_VPH
- J3 pad 3: V+ -> /_V+
- J3 pad 5: VDO -> /_VDO
Routing:
- net 0PH: track 0.00 -> 151.7 mm, vias 0 -> 30
- net VCC: track 0.00 -> 145.6 mm, vias 0 -> 5
- net VPH: track 4.78 -> 139.3 mm, vias 0 -> 4
- net V+: track 4.61 -> 128.2 mm, vias 0 -> 7
- net VDO: track 4.78 -> 120.5 mm, vias 0 -> 4
- net 0V+: track 0.00 -> 80.9 mm, vias 0 -> 17
- net MP: track 0.00 -> 80.2 mm, vias 0 -> 2
- net MPARSER: track 0.00 -> 75.6 mm, vias 0 -> 2
- net SCK: track 0.00 -> 73.5 mm, vias 0 -> 3
- net MZ: track 0.00 -> 70.7 mm, vias 0 -> 2
- net 5VPH: track 4.78 -> 75.1 mm, vias 0 -> 3
- net MISO: track 0.00 -> 41.9 mm, vias 0 -> 2
- net /_VDO: track 0.00 -> 39.1 mm
- net MOSI: track 0.00 -> 37.0 mm, vias 0 -> 2
- net MREL2: track 0.00 -> 36.6 mm, vias 0 -> 2
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- added copper zone on F.Cu, net 0PH
- added copper zone on F.Cu, net 0V+
Other:
- board size 80 x 80 mm -> 80 x 90 mm

Commit message: Silkscreen fixes.
Parts:
- added REF**: OSHW-Logo2_14.6x12mm_SilkScreen, Symbol:OSHW-Logo2_14.6x12mm_SilkScreen, F.Cu at (179.8, 63.2)
- JP1: moved to F.Cu
- moved TP1 49.2 mm to (203.1, 105.8)
- turned JP1 to 180 degrees
Other:
- board text added: "0PH"
- board text added: "0V+"
- board text added: "5V"
- board text added: "GND"
- board text added: "MISO"
- board text added: "ML"
- board text added: "MOSI"
- board text added: "MR"
- board text added: "NC"
- board text added: "REL1"
- board text added: "REL2"
- board text added: "RST"
- board text added: "RX"
- board text added: "SCK"
- board text added: "Solari Control v1.0 KMŽ Brno I JH 2023"
- board text added: "TX"
- board text added: "V+"
- board text added: "VCC"
- board text added: "VDO"
- board text added: "VPH"
- board text added: "https://github.com/kmzbrnoI/solari-control"
- board text added: "⏚"

Commit message: Add test points for remaining grounds.
Parts:
- added TP2: TP, TestPoint:TestPoint_Loop_D3.50mm_Drill1.4mm_Beaded, F.Cu at (213.1, 57.1)
- added TP3: TP, TestPoint:TestPoint_Loop_D3.50mm_Drill1.4mm_Beaded, F.Cu at (144.3, 58.9)
Changed lines of the file:
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@@
     )
   )
+  (footprint "TestPoint:TestPoint_Loop_D3.50mm_Drill1.4mm_Beaded" (layer "F.Cu")
+    (at 144.272 58.928)
+    (descr "wire loop with bead as test point, loop diameter 3.5mm, hole diameter 1.4mm")
+    (tags "test point wire loop bead")
+    (property "Sheetfile" "solari-control.kicad_sch")
+    (property "Sheetname" "")
+    (attr through_hole)
+    (fp_text reference "TP3" (at 0 3.048) (layer "F.SilkS")
+      (effects (font (size 1 1) (thickness 0.15)))
+    )
+    (fp_text value "TP" (at 0 -2.8) (layer "F.Fab")
+      (effects (font (size 1 1) (thickness 0.15)))
+    )
+    (fp_text user "${REFERENCE}" (at 0.7 2.5) (layer "F.Fab")
+      (effects (font (size 1 1) (thickness 0.15)))
+    )
+    (fp_circle (center 0 0) (end 1.8 0) (layer "F.SilkS") (width 0.12) (fill none))
+    (fp_circle (center 0 0) (end 2.1 0) (layer "F.CrtYd") (width 0.05) (fill none))
+    (fp_line (start -1.6 -0.3) (end -1.6 0.3) (layer "F.Fab") (width 0.12))
+    (fp_line (start 1.6 0.3) (end 1.6 -0.3) (layer "F.Fab") (width 0.12))
+    (fp_line (start 1.6 -0.3) (end -1.6 -0.3) (layer "F.Fab") (width 0.12))
+    (fp_line (start -1.6 0.3) (end 1.6 0.3) (layer "F.Fab") (width 0.12))
+    (fp_circle (center 0 0) (end 1.5 0) (layer "F.Fab") (width 0.12) (fill none))
+    (pad "1" thru_hole circle (at 0 0) (size 2.8 2.8) (drill 1.4) (layers *.Cu *.Mask)
+      (net 2 "0PH") (pinfunction "1") (pintype "passive"))
+    (model "${KICAD6_3DMODEL_DIR}/TestPoint.3dshapes/TestPoint_Loop_D3.50mm_Drill1.4mm_Beaded.wrl"
+      (offset (xyz 0 0 0))
+      (scale (xyz 1 1 1))
+      (rotate (xyz 0 0 0))
+    )
+  )
   (footprint "Resistor_SMD:R_0805_2012Metric_Pad1.20x1.40mm_HandSolder" (layer "F.Cu")
     (at 154.194 92.71 180)
@@
     )
   )
+  (footprint "TestPoint:TestPoint_Loop_D3.50mm_Drill1.4mm_Beaded" (layer "F.Cu")
+    (at 213.106 57.15)
+    (descr "wire loop with bead as test point, loop diameter 3.5mm, hole diameter 1.4mm")
+    (tags "test point wire loop bead")
+    (property "Sheetfile" "solari-control.kicad_sch")
+    (property "Sheetname" "")
+    (attr through_hole)
+    (fp_text reference "TP2" (at 0 3.048) (layer "F.SilkS")
+      (effects (font (size 1 1) (thickness 0.15)))
+    )
+    (fp_text value "TP" (at 0 -2.8) (layer "F.Fab")
+      (effects (font (size 1 1) (thickness 0.15)))
+    )
+    (fp_text user "${REFERENCE}" (at 0.7 2.5) (layer "F.Fab")
+      (effects (font (size 1 1) (thickness 0.15)))
+    )
+    (fp_circle (center 0 0) (end 1.8 0) (layer "F.SilkS") (width 0.12) (fill none))
+    (fp_circle (center 0 0) (end 2.1 0) (layer "F.CrtYd") (width 0.05) (fill none))
+    (fp_line (start 1.6 0.3) (end 1.6 -0.3) (layer "F.Fab") (width 0.12))
+    (fp_line (start -1.6 0.3) (end 1.6 0.3) (layer "F.Fab") (width 0.12))
+    (fp_line (start -1.6 -0.3) (end -1.6 0.3) (layer "F.Fab") (width 0.12))
+    (fp_line (start 1.6 -0.3) (end -1.6 -0.3) (layer "F.Fab") (width 0.12))
+    (fp_circle (center 0 0) (end 1.5 0) (layer "F.Fab") (width 0.12) (fill none))
+    (pad "1" thru_hole circle (at 0 0) (size 2.8 2.8) (drill 1.4) (layers *.Cu *.Mask)
+      (net 4 "0V+") (pinfunction "1") (pintype "passive"))
+    (model "${KICAD6_3DMODEL_DIR}/TestPoint.3dshapes/TestPoint_Loop_D3.50mm_Drill1.4mm_Beaded.wrl"
+      (offset (xyz 0 0 0))
+      (scale (xyz 1 1 1))
+      (rotate (xyz 0 0 0))
+    )
+  )
   (footprint "Capacitor_SMD:C_0805_2012Metric_Pad1.18x1.45mm_HandSolder" (layer "F.Cu")
     (at 145.796 114.808)
@@
     (property "Sheetname" "")
     (attr smd)
-    (fp_text reference "R12" (at -3.397 0.016) (layer "B.SilkS")
+    (fp_text reference "R12" (at -3.397 -0.619) (layer "B.SilkS")
       (effects (font (size 1 1) (thickness 0.15)) (justify mirror))
     )
@@
     (property "Sheetname" "")
     (attr smd)
-    (fp_text reference "Q3" (at 0 -2.508 90) (layer "B.SilkS")
+    (fp_text reference "Q3" (at -0.905 -2.508 90) (layer "B.SilkS")
       (effects (font (size 1 1) (thickness 0.15)) (justify mirror))
     )
@@
     (effects (font (size 1 1) (thickness 0.15)) (justify left))
   )
+  (gr_text "0PH" (at 144.272 55.88) (layer "F.SilkS")
+    (effects (font (size 1 1) (thickness 0.15)))
+  )
   (gr_text "V+" (at 195.58 118.618 90) (layer "F.SilkS")
     (effects (font (size 1.5 1.5) (thickness 0.2)) (justify left))
@@
     (effects (font (size 1 1) (thickness 0.15)) (justify right))
   )
+  (gr_text "0V+" (at 213.106 54.102) (layer "F.SilkS")
+    (effects (font (size 1 1) (thickness 0.15)))
+  )
   (segment (start 151.638 69.088) (end 149.622 67.072) (width 0.4) (layer "F.Cu") (net 1))
