File: solari-control.kicad_pcb (KiCad board)
At the start: 2 copper layers, 80 x 90 mm, 112 parts, among them J1 Conn_01x04, J2 A5081WV-5P, J3 A5081WR-5P, J4 AVR-ISP-6, J5 DIL8, J6 Conn_01x04, Q1 AO3401A, Q10 AO3400A, Q11 AO3401A, Q12 AO3400A, Q2 AO3400A, Q3 AO3401A, Q4 AO3400A, Q5 AO3401A, Q6 AO3401A, Q7 AO3401A, Q8 AO3401A, Q9 AO3401A, U1 VO0631T, U10 PC817, U11 PC817, U12 AMS1117-3.3, U2 L78L05_SOT89, U3 VO0631T, U4 PC817, U5 PC817, U6 VO0631T, U7 ATmega328P-A, U8 VO0631T, U9 VO0631T, Y1 14.7456 MHz

Commit message: Sch: use galvanic separation on UART interface.
Other:
- board text added: "Beware: 3V3 logic!"
- board text added: "Disconnect EX for programming"
- board text added: "EX"
Changed lines of the file:
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@@
     (property "Sheetname" "")
     (attr through_hole)
-    (fp_text reference "J4" (at 1.27 -2.33 -270) (layer "F.SilkS")
+    (fp_text reference "J4" (at 1.275 7.605 -270) (layer "F.SilkS")
       (effects (font (size 1 1) (thickness 0.15)))
     )
@@
   (gr_line (start 150.876 65.024) (end 150.876 67.183) (layer "B.SilkS") (width 0.15))
   (gr_line (start 144.272 62.484) (end 156.972 62.484) (layer "B.SilkS") (width 0.15))
+  (gr_line (start 203.454 97.028) (end 204.724 97.028) (layer "F.SilkS") (width 0.15))
+  (gr_line (start 203.454 86.614) (end 203.454 97.028) (layer "F.SilkS") (width 0.15))
+  (gr_line (start 163.83 94.996) (end 172.466 94.996) (layer "F.SilkS") (width 0.15))
+  (gr_line (start 204.724 86.614) (end 203.454 86.614) (layer "F.SilkS") (width 0.15))
+  (gr_line (start 163.83 99.568) (end 163.83 94.996) (layer "F.SilkS") (width 0.15))
+  (gr_line (start 172.466 94.996) (end 172.466 99.568) (layer "F.SilkS") (width 0.15))
   (gr_arc (start 140 44) (mid 141.171573 41.171573) (end 144 40) (layer "Edge.Cuts") (width 0.1))
   (gr_line (start 216 40) (end 144 40) (layer "Edge.Cuts") (width 0.1))
@@
   (gr_line (start 220 126) (end 220 44) (layer "Edge.Cuts") (width 0.1))
   (gr_line (start 140 44) (end 140 126) (layer "Edge.Cuts") (width 0.1))
+  (gr_text "Beware:\n3V3 logic!" (at 201.422 91.694 90) (layer "F.SilkS")
+    (effects (font (size 1 1) (thickness 0.15)))
+  )
   (gr_text "Solari Control\nv1.0\nKMŽ Brno I JH 2023" (at 179.705 80.645) (layer "F.SilkS")
     (effects (font (size 2 2) (thickness 0.25)))
@@
     (effects (font (size 1 1) (thickness 0.15)) (justify left))
   )
+  (gr_text "Disconnect EX\nfor programming" (at 172.72 104.902) (layer "F.SilkS")
+    (effects (font (size 0.8 0.8) (thickness 0.1)) (justify left))
+  )
   (gr_text "GND" (at 165.608 108.966 90) (layer "F.SilkS")
     (effects (font (size 1 1) (thickness 0.15)) (justify right))
@@
     (effects (font (size 1 1) (thickness 0.15)) (justify right))
   )
+  (gr_text "EX" (at 191.008 48.006 90) (layer "F.SilkS")
+    (effects (font (size 1 1) (thickness 0.15)))
+  )
   (gr_text "NC" (at 205.994 45.974 90) (layer "F.SilkS")
     (effects (font (size 1 1) (thickness 0.15)) (justify right))
@@
     (effects (font (size 1 1) (thickness 0.15)) (justify right))
   )
+  (gr_text "Beware:\n3V3 logic!" (at 168.148 96.774) (layer "F.SilkS")
+    (effects (font (size 1 1) (thickness 0.15)))
+  )
   (gr_text "VDO" (at 198.374 45.974 90) (layer "F.SilkS")

Commit message: Wire new changes on PCB.
Parts:
- removed C14: 10u, Capacitor_SMD:C_0805_2012Metric_Pad1.18x1.45mm_HandSolder
- removed JP2: Jumper_3_Open, Connector_PinHeader_2.54mm:PinHeader_1x03_P2.54mm_Vertical
- removed U12: AMS1117-3.3, Package_TO_SOT_SMD:SOT-223-3_TabPin2
- added C16: 100n, Capacitor_SMD:C_0805_2012Metric_Pad1.18x1.45mm_HandSolder, B.Cu at (198.1, 93.5)
- added C17: 100n, Capacitor_SMD:C_0805_2012Metric_Pad1.18x1.45mm_HandSolder, B.Cu at (200.2, 104.9)
- added U13: ADuM1201AR, Package_SO:SOIC-8_3.9x4.9mm_P1.27mm, B.Cu at (202.2, 97.0)
- C2: value 22u/25V -> 22u
- JP1: value J2O -> Jumper_2_Open
- moved JP1 50.7 mm to (158.8, 108.5)
- moved TP1 44.5 mm to (159.5, 96.5)
- moved J1 16.2 mm to (198.9, 108.2), turned to 90 degrees
- moved D1 12.6 mm to (205.2, 104.1), turned to 180 degrees
- moved C2 6.65 mm to (152.4, 114.3), turned to 0 degrees
- moved C10 6.10 mm to (189.3, 107.2)
- moved C11 6.10 mm to (184.8, 107.2)
- moved Y1 6.10 mm to (184.6, 103.4)
Connections:
- net 5V renamed /5V
- C2 pad 1: Net-(C2-Pad1) -> VCC
- D1 pad 2: GND -> /GNDU
- D1 pad 4: TX -> /TXU
- D1 pad 6: RX -> /RXU
- F1 pad 2: Net-(C2-Pad1) -> VCC
- J1 pad 1: Net-(J1-Pad1) -> /VCCU
- J1 pad 2: RX -> /RXU
- J1 pad 3: TX -> /TXU
- J1 pad 4: GND -> /GNDU
- JP1 pad 2: Net-(J1-Pad1) -> Net-(J4-Pad2)
Routing:
- net /5V: track 22.7 -> 5.65 mm, vias 1 -> 0
- net VCC: track 145.6 -> 131.4 mm, vias 5 -> 6
- net /RXU: track 0.00 -> 12.7 mm
- net /TXU: track 0.00 -> 11.5 mm
- net RX: track 36.6 -> 25.8 mm, vias 1 -> 2
- net Net-(C2-Pad1): track 9.70 -> 0.00 mm
- net /VCCU: track 0.00 -> 9.28 mm
- net TX: track 34.5 -> 26.1 mm, vias 1 -> 2
- net Net-(C10-Pad1): track 16.2 -> 11.4 mm
- net Net-(J1-Pad1): track 4.07 -> 0.00 mm
- net Net-(C11-Pad1): track 10.9 -> 7.67 mm
- net MREL2: track 36.6 -> 35.3 mm
- net MREL1: track 31.7 -> 30.6 mm
- net GND: vias 37 -> 39
- net /GNDU: vias 0 -> 6
- added copper zone on B.Cu, net /GNDU
- added copper zone on F.Cu, net /GNDU
Other:
- board text added: "Disconnect ML before connecting!"
- board text removed: "Beware: 3V3 logic!"
