File: pcb/solari-control.kicad_sch (KiCad schematic)
At the start: 111 parts, among them J1 Conn_01x04, J2 A5081WV-5P, J3 A5081WR-5P, J4 AVR-ISP-6, J5 DIL8, J6 Conn_01x04, Q1 AO3401A, Q10 AO3400A, Q11 AO3401A, Q12 AO3400A, Q2 AO3400A, Q3 AO3401A, Q4 AO3400A, Q5 AO3401A, Q6 AO3401A, Q7 AO3401A, Q8 AO3401A, Q9 AO3401A, U1 VO0631T, U10 PC817, U11 PC817, U13 ADuM1201AR, U2 L78L05_SOT89, U3 VO0631T, U4 PC817, U5 PC817, U6 VO0631T, U7 ATmega328P-A, U8 VO0631T, U9 VO0631T, Y1 14.7456 MHz

Commit message: Add GPIO for all hardware.
Parts:
- Q10, Q12, Q2, Q4: value AO3400A -> 2N7002
- Q11, Q9: value AO3401A -> BSS84A
- Q5, Q6: value AO3401A -> BSS83
Other:
- note added: "Alternative: BSS138"
- note added: "BC857"
- note added: "Ugs > 15V Uds > 15V"
- note added: "Ugs > 24V Uds > 24V"
Changed lines of the file:
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@@
     (effects (font (size 1.27 1.27)) (justify right bottom))
+  )
+  (text "BC857" (at 111.125 269.24 0)
+    (effects (font (size 1.27 1.27)) (justify left bottom))
   )
   (text "15V" (at 112.395 43.18 0)
@@
   (text ">" (at 33.02 128.905 180)
     (effects (font (size 1.27 1.27)) (justify right bottom))
+  )
+  (text "Ugs > 24V\nUds > 24V" (at 81.28 242.57 0)
+    (effects (font (size 1.27 1.27)) (justify left bottom))
   )
   (text "From power supply\nFlap unit (MR)\nV+ ~ outputs\nV+ = 5V\nVDO = VR = 24V"
@@
     (effects (font (size 1.27 1.27)) (justify right bottom))
   )
+  (text "Ugs > 15V\nUds > 15V" (at 62.865 73.025 180)
+    (effects (font (size 1.27 1.27)) (justify right bottom))
+  )
   (text "<" (at 62.865 141.605 180)
     (effects (font (size 1.27 1.27)) (justify right bottom))
@@
   )
   (text ">" (at 62.865 133.985 180)
+    (effects (font (size 1.27 1.27)) (justify right bottom))
+  )
+  (text "Alternative:\nBSS138" (at 80.645 85.09 180)
     (effects (font (size 1.27 1.27)) (justify right bottom))
   )
@@
     (in_bom yes) (on_board yes)
     (property "Reference" "Q11" (id 0) (at 114.3 263.525 0))
-    (property "Value" "AO3401A" (id 1) (at 114.3 265.43 0))
+    (property "Value" "BSS84A" (id 1) (at 114.3 265.43 0))
     (property "Footprint" "Package_TO_SOT_SMD:SOT-23" (id 2) (at 106.68 259.08 0)
       (effects (font (size 1.27 1.27) italic) (justify left) hide)
@@
       (effects (font (size 1.27 1.27)) (justify right))
     )
-    (property "Value" "AO3401A" (id 1) (at 111.125 250.825 0))
+    (property "Value" "BSS84A" (id 1) (at 111.125 250.825 0))
     (property "Footprint" "Package_TO_SOT_SMD:SOT-23" (id 2) (at 103.505 244.475 0)
       (effects (font (size 1.27 1.27) italic) (justify left) hide)
@@
     (in_bom yes) (on_board yes)
     (property "Reference" "Q6" (id 0) (at 103.505 111.76 0))
-    (property "Value" "AO3401A" (id 1) (at 113.03 116.205 0)
+    (property "Value" "BSS83" (id 1) (at 113.03 116.205 0)
       (effects (font (size 1.27 1.27)) hide)
     )
@@
       (effects (font (size 1.27 1.27)) (justify right))
     )
-    (property "Value" "AO3400A" (id 1) (at 85.725 245.745 0)
+    (property "Value" "2N7002" (id 1) (at 85.725 245.745 0)
       (effects (font (size 1.27 1.27)) (justify right))
     )
@@
       (effects (font (size 1.27 1.27)) (justify left))
     )
-    (property "Value" "AO3401A" (id 1) (at 91.44 102.235 0)
+    (property "Value" "BSS83" (id 1) (at 91.44 102.235 0)
       (effects (font (size 1.27 1.27)) (justify left))
     )
@@
       (effects (font (size 1.27 1.27)) (justify left))
     )
-    (property "Value" "AO3400A" (id 1) (at 84.9631 264.3628 0)
+    (property "Value" "2N7002" (id 1) (at 84.9631 264.3628 0)
       (effects (font (size 1.27 1.27)) (justify left) hide)
     )
@@
       (effects (font (size 1.27 1.27)) (justify left))
     )
-    (property "Value" "AO3400A" (id 1) (at 83.6931 81.4828 0)
+    (property "Value" "2N7002" (id 1) (at 83.6931 81.4828 0)
       (effects (font (size 1.27 1.27)) (justify left) hide)
     )
@@
       (effects (font (size 1.27 1.27)) (justify right))
     )
-    (property "Value" "AO3400A" (id 1) (at 84.455 62.865 0)
+    (property "Value" "2N7002" (id 1) (at 84.455 62.865 0)
       (effects (font (size 1.27 1.27)) (justify right))
     )
@@
     )
     (path "/af4b59b3-7d09-49d9-adde-1ec7817e4783"
-      (reference "Q2") (unit 1) (value "AO3400A") (footprint "Package_TO_SOT_SMD:SOT-23")
+      (reference "Q2") (unit 1) (value "2N7002") (footprint "Package_TO_SOT_SMD:SOT-23")
     )
     (path "/8899d456-9adf-4924-89a1-55b4ecc5e79e"
@@
     )
     (path "/a22b599a-ef25-4281-a890-6244b7625980"
-      (reference "Q4") (unit 1) (value "AO3400A") (footprint "Package_TO_SOT_SMD:SOT-23")
+      (reference "Q4") (unit 1) (value "2N7002") (footprint "Package_TO_SOT_SMD:SOT-23")
     )
     (path "/61407c9e-ed29-4d9a-ae02-49b50e71759c"
-      (reference "Q5") (unit 1) (value "AO3401A") (footprint "Package_TO_SOT_SMD:SOT-23")
+      (reference "Q5") (unit 1) (value "BSS83") (footprint "Package_TO_SOT_SMD:SOT-23")
     )
     (path "/48774498-7a00-49d8-b20d-bfbc57f17aec"
-      (reference "Q6") (unit 1) (value "AO3401A") (footprint "Package_TO_SOT_SMD:SOT-23")
+      (reference "Q6") (unit 1) (value "BSS83") (footprint "Package_TO_SOT_SMD:SOT-23")
     )
     (path "/1dba0a9f-c794-4358-a346-764c5c892fb6"
@@
     )
     (path "/3b2d0e03-eed8-4245-a76e-b4b16405008b"
-      (reference "Q9") (unit 1) (value "AO3401A") (footprint "Package_TO_SOT_SMD:SOT-23")
+      (reference "Q9") (unit 1) (value "BSS84A") (footprint "Package_TO_SOT_SMD:SOT-23")
     )
     (path "/5a9a9c0a-0e78-46d1-864f-6cc4d151af3e"
-      (reference "Q10") (unit 1) (value "AO3400A") (footprint "Package_TO_SOT_SMD:SOT-23")
+      (reference "Q10") (unit 1) (value "2N7002") (footprint "Package_TO_SOT_SMD:SOT-23")
     )
     (path "/22785a07-7ecc-44c9-9fdf-71a04c9260de"
-      (reference "Q11") (unit 1) (value "AO3401A") (footprint "Package_TO_SOT_SMD:SOT-23")
+      (reference "Q11") (unit 1) (value "BSS84A") (footprint "Package_TO_SOT_SMD:SOT-23")
     )
     (path "/74aa41fe-b5ab-41ad-a421-268696955e25"
-      (reference "Q12") (unit 1) (value "AO3400A") (footprint "Package_TO_SOT_SMD:SOT-23")
+      (reference "Q12") (unit 1) (value "2N7002") (footprint "Package_TO_SOT_SMD:SOT-23")
     )
     (path "/c2810aa4-bb83-4bae-9c63-daff9cb6b16d"

Commit message: Use bipolar resistors for relay control.
Ugs must be >= 30 V, this is unachivable with MOSFETs in SOT23.
Parts:
- removed R39, R42: 10k, Resistor_SMD:R_0805_2012Metric_Pad1.20x1.40mm_HandSolder, symbol Device:R
- Q10, Q12: value 2N7002 -> BC847; symbol Transistor_FET:AO3400A -> Transistor_BJT:BC847
- Q11, Q9: value BSS84A -> BC857; symbol Transistor_FET:AO3401A -> Transistor_BJT:BC857
- R40, R44: value 100R -> 10k
Connections:
- net 0V+: no longer R43.1, R46.1
- net at Q12.1 (B), R46.2: no longer Q11.3 (D)
- net at Q9.3 (C), R43.2: no longer Q10.1 (G)
- new net: Q11.3 (C), R46.1
- new net: Q10.1 (B), R43.1
Other:
- note added: "From power supply Flap unit (MR) V+ ~ outputs V+ = 5V VDO = VR = 24-30V"
- note added: "Ugs > 30V Uds > 30V"
- note removed: "BC857"
- note removed: "From power supply Flap unit (MR) V+ ~ outputs V+ = 5V VDO = VR = 24V"
- note removed: "Ugs > 24V Uds > 24V"
- moved on the sheet: R43, R46

Commit message: Use lower pullups on DATOT & CLOCKT for faster edges.
Parts:
- R22, R24: value 10k -> 2k2
Changed lines of the file:
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@@
       (effects (font (size 1.27 1.27)) (justify right))
     )
-    (property "Value" "10k" (id 1) (at 116.967 144.5772 0)
+    (property "Value" "2k2" (id 1) (at 116.967 144.5772 0)
       (effects (font (size 1.27 1.27)) (justify right))
     )
@@
       (effects (font (size 1.27 1.27)) (justify right))
     )
-    (property "Value" "10k" (id 1) (at 123.317 135.0522 0)
+    (property "Value" "2k2" (id 1) (at 123.317 135.0522 0)
       (effects (font (size 1.27 1.27)) (justify right))
     )
@@
     )
     (path "/1ad690a0-86ab-4bd1-bd9c-673cbcd9a07c"
-      (reference "R22") (unit 1) (value "10k") (footprint "Resistor_SMD:R_0805_2012Metric_Pad1.20x1.40mm_HandSolder")
+      (reference "R22") (unit 1) (value "2k2") (footprint "Resistor_SMD:R_0805_2012Metric_Pad1.20x1.40mm_HandSolder")
     )
     (path "/2a9084b9-0e9b-4b1a-8b73-32228c17c58c"
@@
     )
     (path "/121d6c89-6ff3-48fb-a255-6ef24a424e58"
-      (reference "R24") (unit 1) (value "10k") (footprint "Resistor_SMD:R_0805_2012Metric_Pad1.20x1.40mm_HandSolder")
+      (reference "R24") (unit 1) (value "2k2") (footprint "Resistor_SMD:R_0805_2012Metric_Pad1.20x1.40mm_HandSolder")
     )
     (path "/8d833850-893e-4165-9d69-3891a84665c3"

Commit message: PCB: tweak fast signal resistors, use bipolar transistors for fast signals.
Parts:
- added R39: 470R, Resistor_SMD:R_0805_2012Metric_Pad1.20x1.40mm_HandSolder, symbol Device:R
- Q3: value AO3401A -> BC857; symbol Transistor_FET:AO3401A -> Transistor_BJT:BC857
- Q4: symbol Transistor_FET:AO3400A -> Transistor_BJT:BC847
- R1, R7: value 10k -> 2k2
- R10: value 100R -> 470R
- R12, R8: value 10k -> 100R
Connections:
- net at Q4.1 (B), R12.2: now also R39.1; no longer Q3.3 (D)
- new net: Q3.3 (C), R39.2
Other:
- note added: "Close resistor for fast transitions"
Changed lines of the file:
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@@
     (stroke (width 0) (type default) (color 0 0 0 0))
   )
+  (wire (pts (xy 106.045 83.185) (xy 107.95 83.185))
+    (stroke (width 0) (type default) (color 0 0 0 0))
+  )
   (wire (pts (xy 274.32 52.705) (xy 276.86 52.705))
     (stroke (width 0) (type default) (color 0 0 0 0))
@@
     (stroke (width 0) (type default) (color 0 0 0 0))
   )
-  (wire (pts (xy 95.25 83.185) (xy 107.95 83.185))
+  (wire (pts (xy 95.25 83.185) (xy 98.425 83.185))
     (stroke (width 0) (type default) (color 0 0 0 0))
   )
@@
     (effects (font (size 1.27 1.27)) (justify right bottom))
   )
-  (text "Alternative:\nBSS138" (at 80.645 85.09 180)
+  (text "Alternative:\nBSS138" (at 108.585 55.245 180)
     (effects (font (size 1.27 1.27)) (justify right bottom))
   )
+  (text "Close resistor\nfor fast transitions" (at 109.855 88.265 0)
+    (effects (font (size 1.27 1.27)) (justify left bottom))
+  )
   (text "S = inputs\nT = outputs" (at 37.465 149.86 0)
     (effects (font (size 1.27 1.27)) (justify left bottom))
@@
     (in_bom yes) (on_board yes)
     (property "Reference" "R10" (id 0) (at 125.095 82.55 90))
-    (property "Value" "100R" (id 1) (at 125.095 80.645 90))
+    (property "Value" "470R" (id 1) (at 125.095 80.645 90))
     (property "Footprint" "Resistor_SMD:R_0805_2012Metric_Pad1.20x1.40mm_HandSolder" (id 2) (at 125.095 76.327 90)
       (effects (font (size 1.27 1.27)) hide)
@@
   (symbol (lib_id "Device:R") (at 95.25 86.995 180) (unit 1)
     (in_bom yes) (on_board yes)
-    (property "Reference" "R12" (id 0) (at 97.155 88.265 0)
-      (effects (font (size 1.27 1.27)) (justify right))
+    (property "Reference" "R12" (id 0) (at 93.345 86.36 0)
+      (effects (font (size 1.27 1.27)) (justify left))
     )
-    (property "Value" "10k" (id 1) (at 97.155 86.36 0)
-      (effects (font (size 1.27 1.27)) (justify right))
+    (property "Value" "100R" (id 1) (at 93.345 88.265 0)
+      (effects (font (size 1.27 1.27)) (justify left))
     )
     (property "Footprint" "Resistor_SMD:R_0805_2012Metric_Pad1.20x1.40mm_HandSolder" (id 2) (at 97.028 86.995 90)
@@
     (in_bom yes) (on_board yes)
     (property "Reference" "R8" (id 0) (at 114.3 75.565 90))
-    (property "Value" "10k" (id 1) (at 114.3 70.8461 90))
+    (property "Value" "100R" (id 1) (at 114.3 70.8461 90))
     (property "Footprint" "Resistor_SMD:R_0805_2012Metric_Pad1.20x1.40mm_HandSolder" (id 2) (at 114.3 74.803 90)
       (effects (font (size 1.27 1.27)) hide)
@@
     (pin "2")
   )
-  (symbol (lib_id "Transistor_FET:AO3401A") (at 110.49 78.105 180) (unit 1)
+  (symbol (lib_id "Transistor_BJT:BC857") (at 110.49 78.105 180) (unit 1)
     (in_bom yes) (on_board yes)
-    (property "Reference" "Q3" (id 0) (at 113.03 80.645 0))
-    (property "Value" "AO3401A" (id 1) (at 113.03 82.55 0))
+    (property "Reference" "Q3" (id 0) (at 105.41 76.835 0)
+      (effects (font (size 1.27 1.27)) (justify left))
+    )
+    (property "Value" "BC857" (id 1) (at 105.41 79.375 0)
+      (effects (font (size 1.27 1.27)) (justify left))
+    )
     (property "Footprint" "Package_TO_SOT_SMD:SOT-23" (id 2) (at 105.41 76.2 0)
       (effects (font (size 1.27 1.27) italic) (justify left) hide)
     )
-    (property "Datasheet" "http://www.aosmd.com/pdfs/datasheet/AO3401A.pdf" (id 3) (at 110.49 78.105 0)
+    (property "Datasheet" "https://www.onsemi.com/pub/Collateral/BC860-D.pdf" (id 3) (at 110.49 78.105 0)
       (effects (font (size 1.27 1.27)) (justify left) hide)
     )
@@
       (effects (font (size 1.27 1.27)) (justify right))
     )
-    (property "Value" "10k" (id 1) (at 74.93 69.85 0)
+    (property "Value" "2k2" (id 1) (at 74.93 69.85 0)
       (effects (font (size 1.27 1.27)) (justify right))
     )
@@
     (pin "1")
   )
-  (symbol (lib_id "Transistor_FET:AO3400A") (at 88.9 83.185 0) (mirror y) (unit 1)
+  (symbol (lib_id "Transistor_BJT:BC847") (at 88.9 83.185 0) (mirror y) (unit 1)
     (in_bom yes) (on_board yes)
     (property "Reference" "Q4" (id 0) (at 91.44 79.375 0)
@@
       (effects (font (size 1.27 1.27) italic) (justify left) hide)
     )
-    (property "Datasheet" "http://www.aosmd.com/pdfs/datasheet/AO3400A.pdf" (id 3) (at 88.9 83.185 0)
+    (property "Datasheet" "http://www.infineon.com/dgdl/Infineon-BC847SERIES_BC848SERIES_BC849SERIES_BC850SERIES-DS-v01_01-en.pdf?fileId=db3a304314dca389011541d4630a1657" (id 3) (at 88.9 83.185 0)
       (effects (font (size 1.27 1.27)) (justify left) hide)
     )
@@
       (effects (font (size 1.27 1.27)) (justify right))
     )
-    (property "Value" "10k" (id 1) (at 165.608 37.2622 0)
+    (property "Value" "2k2" (id 1) (at 165.608 37.2622 0)
       (effects (font (size 1.27 1.27)) (justify right))
     )
@@
     (pin "1")
   )
+  (symbol (lib_id "Device:R") (at 102.235 83.185 90) (unit 1)
+    (in_bom yes) (on_board yes)
+    (property "Reference" "R39" (id 0) (at 102.235 85.725 90))
+    (property "Value" "470R" (id 1) (at 102.235 87.63 90))
+    (property "Footprint" "Resistor_SMD:R_0805_2012Metric_Pad1.20x1.40mm_HandSolder" (id 2) (at 102.235 84.963 90)
+      (effects (font (size 1.27 1.27)) hide)
+    )
+    (property "Datasheet" "~" (id 3) (at 102.235 83.185 0)
+      (effects (font (size 1.27 1.27)) hide)
+    )
+    (pin "1")
+    (pin "2")
+  )
   (symbol (lib_id "Device:C") (at 131.445 73.025 0) (mirror y) (unit 1)
     (in_bom yes) (on_board yes)
@@
     )
     (path "/8899d456-9adf-4924-89a1-55b4ecc5e79e"
-      (reference "Q3") (unit 1) (value "AO3401A") (footprint "Package_TO_SOT_SMD:SOT-23")
+      (reference "Q3") (unit 1) (value "BC857") (footprint "Package_TO_SOT_SMD:SOT-23")
     )
     (path "/a22b599a-ef25-4281-a890-6244b7625980"
@@
     )
     (path "/c2810aa4-bb83-4bae-9c63-daff9cb6b16d"
-      (reference "R1") (unit 1) (value "10k") (footprint "Resistor_SMD:R_0805_2012Metric_Pad1.20x1.40mm_HandSolder")
+      (reference "R1") (unit 1) (value "2k2") (footprint "Resistor_SMD:R_0805_2012Metric_Pad1.20x1.40mm_HandSolder")
     )
     (path "/10b327a4-ab34-47c4-9ae9-0d37086e9653"
@@
     )
     (path "/98793b64-96d2-400b-bad0-f545bed1c709"
-      (reference "R7") (unit 1) (value "10k") (footprint "Resistor_SMD:R_0805_2012Metric_Pad1.20x1.40mm_HandSolder")
+      (reference "R7") (unit 1) (value "2k2") (footprint "Resistor_SMD:R_0805_2012Metric_Pad1.20x1.40mm_HandSolder")
     )
     (path "/3ff5e6c2-6c9d-485f-83ad-f18567e6d753"
-      (reference "R8") (unit 1) (value "10k") (footprint "Resistor_SMD:R_0805_2012Metric_Pad1.20x1.40mm_HandSolder")
+      (reference "R8") (unit 1) (value "100R") (footprint "Resistor_SMD:R_0805_2012Metric_Pad1.20x1.40mm_HandSolder")
     )
     (path "/df6a50b3-4015-4e9f-8ca2-b133514dd08e"
@@
     )
     (path "/068ad563-4cbd-47b4-843f-42df19a5ca62"
-      (reference "R10") (unit 1) (value "100R") (footprint "Resistor_SMD:R_0805_2012Metric_Pad1.20x1.40mm_HandSolder")
+      (reference "R10") (unit 1) (value "470R") (footprint "Resistor_SMD:R_0805_2012Metric_Pad1.20x1.40mm_HandSolder")
     )
     (path "/06e9b399-676e-4a21-910c-421c693e7bf2"
@@
     )
     (path "/2f902a55-58d8-42ef-9589-f0ada3121395"
-      (reference "R12") (unit 1) (value "10k") (footprint "Resistor_SMD:R_0805_2012Metric_Pad1.20x1.40mm_HandSolder")
+      (reference "R12") (unit 1) (value "100R") (footprint "Resistor_SMD:R_0805_2012Metric_Pad1.20x1.40mm_HandSolder")
     )
     (path "/03a0a957-054a-454d-bf59-2c0ea20e2ba9"
@@
       (reference "R38") (unit 1) (value "10k") (footprint "Resistor_SMD:R_0805_2012Metric_Pad1.20x1.40mm_HandSolder")
     )
+    (path "/e1c0ef6c-eb94-429a-9988-8216ef3edc2a"
+      (reference "R39") (unit 1) (value "470R") (footprint "Resistor_SMD:R_0805_2012Metric_Pad1.20x1.40mm_HandSolder")
+    )
     (path "/324d318b-4d46-4963-b6de-4bfb2c000209"

Commit message: Fix 'Z' & 'P' pins.
Parts:
- R13, R17: value 10k -> 470R
- R14, R19: value 100R -> 1k
Connections:
- net MP: now also R15.2, U7.1 (PD3); no longer R20.2, U7.2 (PD4)
- net MZ: now also R20.2, U7.2 (PD4); no longer R15.2, U7.1 (PD3)
Changed lines of the file:
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@@
     )
   )
-  (global_label "MP" (shape input) (at 167.005 111.76 0) (fields_autoplaced)
+  (global_label "MZ" (shape input) (at 167.005 111.76 0) (fields_autoplaced)
     (effects (font (size 1.27 1.27)) (justify left))
-    (property "Intersheet References" "${INTERSHEET_REFS}" (id 0) (at 172.1395 111.6806 0)
+    (property "Intersheet References" "${INTERSHEET_REFS}" (id 0) (at 172.0791 111.6806 0)
       (effects (font (size 1.27 1.27)) (justify left) hide)
     )
@@
     )
   )
-  (global_label "MZ" (shape input) (at 254 194.31 180) (fields_autoplaced)
-    (effects (font (size 1.27 1.27)) (justify right))
-    (property "Intersheet References" "${INTERSHEET_REFS}" (id 0) (at 248.9259 194.2306 0)
-      (effects (font (size 1.27 1.27)) (justify right) hide)
-    )
-  )
-  (global_label "MP" (shape input) (at 254 196.85 180) (fields_autoplaced)
-    (effects (font (size 1.27 1.27)) (justify right))
-    (property "Intersheet References" "${INTERSHEET_REFS}" (id 0) (at 248.8655 196.7706 0)
+  (global_label "MP" (shape input) (at 254 194.31 180) (fields_autoplaced)
+    (effects (font (size 1.27 1.27)) (justify right))
+    (property "Intersheet References" "${INTERSHEET_REFS}" (id 0) (at 248.8655 194.2306 0)
+      (effects (font (size 1.27 1.27)) (justify right) hide)
+    )
+  )
+  (global_label "MZ" (shape input) (at 254 196.85 180) (fields_autoplaced)
+    (effects (font (size 1.27 1.27)) (justify right))
+    (property "Intersheet References" "${INTERSHEET_REFS}" (id 0) (at 248.9259 196.7706 0)
       (effects (font (size 1.27 1.27)) (justify right) hide)
     )
@@
     )
   )
-  (global_label "MZ" (shape input) (at 167.005 101.6 0) (fields_autoplaced)
+  (global_label "MP" (shape input) (at 167.005 101.6 0) (fields_autoplaced)
     (effects (font (size 1.27 1.27)) (justify left))
-    (property "Intersheet References" "${INTERSHEET_REFS}" (id 0) (at 172.0791 101.5206 0)
+    (property "Intersheet References" "${INTERSHEET_REFS}" (id 0) (at 172.1395 101.5206 0)
       (effects (font (size 1.27 1.27)) (justify left) hide)
     )
@@
     (in_bom yes) (on_board yes)
     (property "Reference" "R13" (id 0) (at 100.33 99.06 90))
-    (property "Value" "10k" (id 1) (at 100.33 94.3411 90))
+    (property "Value" "470R" (id 1) (at 100.33 94.3411 90))
     (property "Footprint" "Resistor_SMD:R_0805_2012Metric_Pad1.20x1.40mm_HandSolder" (id 2) (at 100.33 98.298 90)
       (effects (font (size 1.27 1.27)) hide)
@@
     (in_bom yes) (on_board yes)
     (property "Reference" "R17" (id 0) (at 113.03 109.22 90))
-    (property "Value" "10k" (id 1) (at 113.03 104.5011 90))
+    (property "Value" "470R" (id 1) (at 113.03 104.5011 90))
     (property "Footprint" "Resistor_SMD:R_0805_2012Metric_Pad1.20x1.40mm_HandSolder" (id 2) (at 113.03 108.458 90)
       (effects (font (size 1.27 1.27)) hide)
@@
     (in_bom yes) (on_board yes)
     (property "Reference" "R19" (id 0) (at 125.095 116.205 90))
-    (property "Value" "100R" (id 1) (at 125.095 114.3 90))
+    (property "Value" "1k" (id 1) (at 125.095 114.3 90))
     (property "Footprint" "Resistor_SMD:R_0805_2012Metric_Pad1.20x1.40mm_HandSolder" (id 2) (at 125.095 109.982 90)
       (effects (font (size 1.27 1.27)) hide)
@@
     (in_bom yes) (on_board yes) (fields_autoplaced)
     (property "Reference" "R14" (id 0) (at 125.095 96.8842 90))
-    (property "Value" "100R" (id 1) (at 125.095 99.4211 90))
+    (property "Value" "1k" (id 1) (at 125.095 99.4211 90))
     (property "Footprint" "Resistor_SMD:R_0805_2012Metric_Pad1.20x1.40mm_HandSolder" (id 2) (at 125.095 103.378 90)
       (effects (font (size 1.27 1.27)) hide)
@@
     )
     (path "/03a0a957-054a-454d-bf59-2c0ea20e2ba9"
-      (reference "R13") (unit 1) (value "10k") (footprint "Resistor_SMD:R_0805_2012Metric_Pad1.20x1.40mm_HandSolder")
+      (reference "R13") (unit 1) (value "470R") (footprint "Resistor_SMD:R_0805_2012Metric_Pad1.20x1.40mm_HandSolder")
     )
     (path "/f97f71a3-782a-4cf0-8404-edd27855faab"
-      (reference "R14") (unit 1) (value "100R") (footprint "Resistor_SMD:R_0805_2012Metric_Pad1.20x1.40mm_HandSolder")
+      (reference "R14") (unit 1) (value "1k") (footprint "Resistor_SMD:R_0805_2012Metric_Pad1.20x1.40mm_HandSolder")
     )
     (path "/8bf71dd6-a42a-4bfe-9da5-755b5bbde6c1"
@@
     )
     (path "/41d9e7bd-9b40-4d62-9500-7a6fdd6750ca"
-      (reference "R17") (unit 1) (value "10k") (footprint "Resistor_SMD:R_0805_2012Metric_Pad1.20x1.40mm_HandSolder")
+      (reference "R17") (unit 1) (value "470R") (footprint "Resistor_SMD:R_0805_2012Metric_Pad1.20x1.40mm_HandSolder")
     )
     (path "/17b9cecb-6e9d-4e95-aa0e-a57e9cb12a47"
@@
     )
     (path "/915a0f58-9261-4e4f-9624-2555c035454f"
-      (reference "R19") (unit 1) (value "100R") (footprint "Resistor_SMD:R_0805_2012Metric_Pad1.20x1.40mm_HandSolder")
+      (reference "R19") (unit 1) (value "1k") (footprint "Resistor_SMD:R_0805_2012Metric_Pad1.20x1.40mm_HandSolder")
     )
     (path "/cd12d761-a612-434b-a2d9-3c857bfa8c67"

Commit message: Update pull-up resistor value.
Parts:
- R7: value 2k2 -> 470R
Changed lines of the file:
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@@
       (effects (font (size 1.27 1.27)) (justify right))
     )
-    (property "Value" "2k2" (id 1) (at 74.93 69.85 0)
+    (property "Value" "470R" (id 1) (at 74.93 69.85 0)
       (effects (font (size 1.27 1.27)) (justify right))
     )
@@
     )
     (path "/98793b64-96d2-400b-bad0-f545bed1c709"
-      (reference "R7") (unit 1) (value "2k2") (footprint "Resistor_SMD:R_0805_2012Metric_Pad1.20x1.40mm_HandSolder")
+      (reference "R7") (unit 1) (value "470R") (footprint "Resistor_SMD:R_0805_2012Metric_Pad1.20x1.40mm_HandSolder")
     )
     (path "/3ff5e6c2-6c9d-485f-83ad-f18567e6d753"

Commit message: Sch: add programming strength note.
Other:
- note added: "A programmer with "strong" outputs must be used to override R11 & R25 pull-ups. J5 shall be disconnected while programming."
